File: Logic-PCB 2/Logi-PCB-2/_autosave-Logi-PCB-2.kicad_sch (KiCad schematic)
At the start: 8 parts, among them Q1 MMBT2222, Q2 MMBT2907A-7-F, SW1 SW_Omron_B3FS, SW1 SW_Push

Commit message: tes
Parts:
- removed R1 (x2): R, symbol Device:R
- removed SW1: SW_Omron_B3FS, symbol Switch:SW_Omron_B3FS
- added R1, R3: R, symbol Device:R
- added SW2: SW_Omron_B3FS, symbol Switch:SW_Omron_B3FS
Connections:
- net +5V: now also R1.1
- net GND: now also R3.2
- net at SW1.2: now also R1.2
- new net: R3.1, SW2.2
