File: Logic-PCB 2/Logi-PCB-2/Logi-PCB-2.kicad_sch (KiCad schematic)
At the start: 55 parts, among them IC1 MC14027BDR2G, IC10 74LVC1G08FW5-7, IC11 MC14027BDR2G, IC12 TMUX4051PWR, IC13 TMUX4051PWR, IC14 TMUX4051PWR, IC15 TMUX4051PWR, IC16 TMUX4051PWR, IC17 TMUX4051PWR, IC18 TMUX4051PWR, IC19 TMUX4051PWR, IC2 LM555CMX_NOPB, IC3 NLV17SZ74USG, IC4 MC14043BDR2G, IC5 MC14027BDR2G, IC6 MC14027BDR2G, IC7 CD4082BM96, IC8 74LVC1G32GV,125, IC9 TMUX4051PWR, Q1 MMBT2222, SW1 SW_Push, SW2 SW_Push, SW3 SW_Push, SW4 SW_Push, SW5 SW_Push, SW6 SW_Push, SW7 SW_Push, SW8 SW_Push

Commit message: PCB 2
Parts:
- removed D6: LED, symbol Device:LED
- removed IC1, IC11, IC5, IC6: MC14027BDR2G, SOIC127P600X175-16N, symbol SamacSys_Parts:MC14027BDR2G
- removed IC10: 74LVC1G08FW5-7, 74LVC1G08FW57, symbol SamacSys_Parts:74LVC1G08FW5-7
- removed IC12, IC13, IC14, IC15, IC16, IC17, IC18, IC19, IC9: TMUX4051PWR, SOP65P640X120-16N, symbol SamacSys_Parts:TMUX4051PWR
- removed IC2: LM555CMX_NOPB, SOIC127P600X175-8N, symbol SamacSys_Parts:LM555CMX_NOPB
- removed IC3: NLV17SZ74USG, SOP50P310X90-8N, symbol SamacSys_Parts:NLV17SZ74USG
- removed IC4: MC14043BDR2G, SOIC127P600X175-16N, symbol SamacSys_Parts:MC14043BDR2G
- removed IC7: CD4082BM96, SOIC127P600X175-14N, symbol SamacSys_Parts:CD4082BM96
- removed IC8: 74LVC1G32GV,125, SOT95P275X110-5N, symbol SamacSys_Parts:74LVC1G32GV,125
- removed Q1: MMBT2222, SamacSys_Parts:SOT95P240X114-3N, symbol SamacSys_Parts:MMBT2222
- removed SW4, SW5, SW6, SW7, SW8: SW_Push, symbol Switch:SW_Push
- added C4: 100n, Capacitor_SMD:C_01005_0402Metric, symbol Device:C
- added C5: 10u, Capacitor_SMD:C_01005_0402Metric, symbol Device:C
- added D10, D11, D12, D7, D8, D9: LED, LED_SMD:LED_0402_1005Metric, symbol Device:LED
- added D6: LSM115JE3_TR13, SamacSys_Parts:DIOM5436X330N, symbol SamacSys_Parts:LSM115JE3_TR13
- added IC1: 74LVC1G74DC-Q100H, SamacSys_Parts:SOP50P310X100-8N, symbol SamacSys_Parts:74LVC1G74DC-Q100H
- added IC10, IC9: SN74LVC1G11MDCKREP, SamacSys_Parts:SOP65P210X110-6N, symbol SamacSys_Parts:SN74LVC1G11MDCKREP
- added IC11, IC12: SN74LVC1G97QDBVRQ1, SamacSys_Parts:SOT95P280X145-6N, symbol SamacSys_Parts:SN74LVC1G97QDBVRQ1
- added IC13, IC14, IC15, IC16, IC17, IC18, IC19, IC20, IC21: TMUX1208QRSVRQ1, SamacSys_Parts:TMUX1208QRSVRQ1, symbol SamacSys_Parts:TMUX1208QRSVRQ1
- added IC2, IC7, IC8: 74HC73D,653, SamacSys_Parts:SOIC127P600X175-14N, symbol SamacSys_Parts:74HC73D,653
- added IC3: TLC555QDRQ1, SamacSys_Parts:SOIC127P600X175-8N, symbol SamacSys_Parts:TLC555QDRQ1
- added IC4, IC5: SN74LVC1G02DBVR, SamacSys_Parts:SOT95P280X145-5N, symbol SamacSys_Parts:SN74LVC1G02DBVR
- added IC6: NCV4274AST33T3G, SamacSys_Parts:SOT230P700X175-4N, symbol SamacSys_Parts:NCV4274AST33T3G
- added J1: CX70M-24P1, SamacSys_Parts:CX70M24P1, symbol SamacSys_Parts:CX70M-24P1
- added R17, R18, R19, R20, R21, R22, R23, R24, R25, R26, R27, R28, R29, R30: 100, Resistor_SMD:R_0402_1005Metric, symbol Device:R
- added S1: JS203011JAQN, SamacSys_Parts:JS203011JAQN, symbol SamacSys_Parts:JS203011JAQN
- added U1: BAT-HLD-001-TR, SamacSys_Parts:BATHLD001TR, symbol SamacSys_Parts:BAT-HLD-001-TR
- C1, C2, C3: footprint (none) -> Capacitor_SMD:C_01005_0402Metric
- D1, D2, D3, D4, D5: footprint (none) -> LED_SMD:LED_0402_1005Metric
- DS1: footprint PSA0811GWA -> SamacSys_Parts:PSA0811GWA
- R1, R2: value R -> 10k; footprint (none) -> Resistor_SMD:R_0402_1005Metric
- R10, R16: value 10k -> 100; footprint (none) -> Resistor_SMD:R_0402_1005Metric
- R11, R3: value 51 -> 100; footprint (none) -> Resistor_SMD:R_0402_1005Metric
- R12, R9: value 10k -> 1k; footprint (none) -> Resistor_SMD:R_0402_1005Metric
- R13, R14, R8: footprint (none) -> Resistor_SMD:R_0402_1005Metric
- R15, R7: value 51 -> 10k; footprint (none) -> Resistor_SMD:R_0402_1005Metric
- R4: value 1k -> 10k; footprint (none) -> Resistor_SMD:R_0402_1005Metric
- R5: value 1k -> 100; footprint (none) -> Resistor_SMD:R_0402_1005Metric
- R6: value 220 -> 100; footprint (none) -> Resistor_SMD:R_0402_1005Metric
- SW1, SW2, SW3: footprint (none) -> SamacSys_Parts:SKPMBHE010
- VR1: footprint 3314J-1 -> SamacSys_Parts:3314J-1
Connections:
- net +3V0: now also C3.1, R16.2, R9.2, SW1.1, IC1.6 (~{RD}), IC1.7 (~{SD}), IC1.8 (VCC), IC10.5 (VCC), IC11.3 (IN0), IC11.5 (VCC), IC12.5 (VCC), IC13.10 (S5), IC13.11 (VDD), IC13.16 (EN), IC13.2 (S1), IC13.3 (S2), IC13.5 (S4), IC14.11 (VDD), IC14.16 (EN), IC14.4 (S3), IC15.11 (VDD), IC15.16 (EN), IC15.2 (S1), IC15.4 (S3), IC16.10 (S5), IC16.11 (VDD), IC16.16 (EN), IC16.2 (S1), IC16.3 (S2), IC17.10 (S5), IC17.11 (VDD), IC17.16 (EN), IC17.2 (S1), IC17.3 (S2), IC17.4 (S3), IC18.11 (VDD), IC18.16 (EN), IC18.4 (S3), IC18.9 (S6), IC19.11 (VDD), IC19.16 (EN), IC19.5 (S4), IC2.2 (1~{R}), IC2.4 (VCC), IC20.11 (VDD), IC20.16 (EN), IC20.9 (S6), IC21.10 (S5), IC21.11 (VDD), IC21.16 (EN), IC21.3 (S2), IC3.4 (RESET), IC3.8 (VDD), IC4.5 (VCC), IC5.5 (VCC), IC7.14 (1J), IC7.2 (1~{R}), IC7.3 (1K), IC7.4 (VCC), IC8.2 (1~{R}), IC8.4 (VCC), IC8.6 (2~{R}), IC9.5 (VCC), S1.8 (NO_2); no longer R1.1, R2.1
- net +5V: now also C4.2, IC6.1 (INPUT), J1.A4 (VBUS_1), J1.A9 (VBUS_2), J1.B4 (VBUS_3), J1.B9 (VBUS_4); no longer C3.1, R4.1
- net Button: now also R15.2, SW3.2, IC7.1 (1~{CP}), IC8.1 (1~{CP}), IC8.5 (2~{CP}); no longer R14.2
- net CLK: now also IC1.1 (CP), IC2.1 (1~{CP}), IC3.3 (OUT)
- net GND: now also DS1.11 (COM_A), DS1.12 (K_DP), R1.1, R15.1, R2.1, R4.1, R7.1, C4.1, C5.2, D10.1 (K), D11.1 (K), D12.1 (K), D7.1 (K), D8.1 (K), D9.1 (K), IC1.4 (GND), IC10.2 (GND), IC11.2 (GND), IC12.1 (IN1), IC12.2 (GND), IC13.12 (GND), IC13.4 (S3), IC13.7 (S8), IC13.8 (S7), IC13.9 (S6), IC14.10 (S5), IC14.12 (GND), IC14.2 (S1), IC14.3 (S2), IC14.5 (S4), IC14.7 (S8), IC14.8 (S7), IC14.9 (S6), IC15.10 (S5), IC15.12 (GND), IC15.3 (S2), IC15.5 (S4), IC15.7 (S8), IC15.8 (S7), IC15.9 (S6), IC16.12 (GND), IC16.4 (S3), IC16.5 (S4), IC16.7 (S8), IC16.8 (S7), IC16.9 (S6), IC17.12 (GND), IC17.5 (S4), IC17.7 (S8), IC17.8 (S7), IC17.9 (S6), IC18.10 (S5), IC18.12 (GND), IC18.2 (S1), IC18.3 (S2), IC18.5 (S4), IC18.7 (S8), IC18.8 (S7), IC19.10 (S5), IC19.12 (GND), IC19.2 (S1), IC19.3 (S2), IC19.4 (S3), IC19.7 (S8), IC19.8 (S7), IC19.9 (S6), IC2.11 (GND), IC20.10 (S5), IC20.12 (GND), IC20.2 (S1), IC20.3 (S2), IC20.4 (S3), IC20.5 (S4), IC20.7 (S8), IC20.8 (S7), IC21.12 (GND), IC21.2 (S1), IC21.4 (S3), IC21.5 (S4), IC21.7 (S8), IC21.8 (S7), IC21.9 (S6), IC3.1 (GND), IC4.3 (GND), IC5.3 (GND), IC6.2 (GROUND_1), IC6.4 (GROUND_2), IC7.11 (GND), IC8.11 (GND), IC9.2 (GND), J1.A1 (GND_1), J1.A12 (GND_2), J1.B1 (GND_3), J1.B12 (GND_4), S1.3 (COM_1), S1.7 (COM_2), U1.3; no longer R10.1, R12.1, R16.1, R9.1
- net at C1.1, VR1.3 (CW): now also IC3.2 (TRIG), IC3.6 (THRES)
- net at VR1.2 (WIPER): now also R12.2; no longer R5.1
- net at R3.2: now also D1.2 (A)
- net Button B: now reaches SW2.2
- net Button B: now also R14.2, R2.2, R8.2, IC2.3 (1K), IC5.1 (A); no longer R9.2
- net at DS1.1 (K_A), DS1.18 (K_B): now also R27.2
- net at DS1.10 (K_E), DS1.15 (K_P), DS1.9 (K_F): now also R30.2
- net at DS1.13 (K_D): now also R29.2
- net at DS1.14 (K_R), DS1.3 (K_K): now also R26.2
- net at DS1.16 (K_C): now also R28.2
- net at DS1.17 (K_N), DS1.7 (K_T): now also R25.2
- net at DS1.2 (K_M), DS1.6 (K_S): now also R24.2
- net at DS1.4 (K_H), DS1.8 (K_G): now also R22.2
- net at DS1.5 (K_U): now also R23.2
- net at D5.2 (A): now also R11.1; no longer R11.2
- net at R5.2: now also IC2.12 (1Q); no longer R4.2
- net at D4.2 (A): now also R10.1; no longer R7.2
- net at R10.2: now also IC4.2 (B), IC5.4 (Y)
- net Button A: now reaches R13.2
- net Button A: now also R1.2, R4.2, R7.2, SW1.2, IC1.2 (D), IC2.14 (1J), IC4.1 (A)
- net at R3.1: now also IC1.5 (Q); no longer D2.2 (A)
- net at C2.1: now also IC3.5 (CONT)
- new net: IC10.3 (B), IC12.3 (IN0), IC13.13 (A2), IC14.13 (A2), IC15.13 (A2), IC16.13 (A2), IC17.13 (A2), IC18.13 (A2), IC19.13 (A2), IC20.13 (A2), IC21.13 (A2), IC7.12 (1Q), IC9.3 (B), R19.2
- new net: IC10.1 (A), IC13.14 (A1), IC14.14 (A1), IC15.14 (A1), IC16.14 (A1), IC17.14 (A1), IC18.14 (A1), IC19.14 (A1), IC20.14 (A1), IC21.14 (A1), IC8.9 (2Q), R20.2
- new net: IC13.15 (A0), IC14.15 (A0), IC15.15 (A0), IC16.15 (A0), IC17.15 (A0), IC18.15 (A0), IC19.15 (A0), IC20.15 (A0), IC21.15 (A0), IC8.12 (1Q), IC9.6 (C), R21.2
- new net: IC18.6 (D), R26.1
- new net: IC15.6 (D), R29.1
- new net: IC3.7 (DISCH), R12.1, R9.1
- new net: D11.2 (A), R20.1
- new net: IC21.6 (D), R23.1
- new net: D12.2 (A), R21.1
- new net: D10.2 (A), R19.1
- new net: D9.2 (A), R18.1
- new net: D2.2 (A), R5.1
- new net: D6.2, U1.1
- new net: IC20.6 (D), R25.1
- new net: IC8.8 (2~{Q}), IC9.1 (A)
- new net: IC11.1 (IN1), IC9.4 (Y)
- new net: IC17.6 (D), R22.1
- new net: IC13.6 (D), R27.1
- new net: IC12.4 (Y), IC8.10 (2K), IC8.7 (2J), R17.2
- new net: IC10.6 (C), IC12.6 (IN2), IC8.13 (1~{Q})
- new net: IC11.4 (Y), IC8.14 (1J), IC8.3 (1K), R18.2
- new net: D7.2 (A), R16.1
- new net: IC14.6 (D), R28.1
- new net: IC16.6 (D), R30.1
- new net: IC4.4 (Y), IC5.2 (B), R11.2
- new net: IC19.6 (D), R24.1
- new net: IC10.4 (Y), IC11.6 (IN2)
- new net: D8.2 (A), R17.1
- new net 3V before switch: C5.1, D6.1, IC6.3 (OUTPUT), S1.4 (NO_1)
- no-connect marks 0 -> 43
Other:
- note added: "16 segment display"
- note added: "3 in AND gate"
- note added: "5V to 3.3V Linear Regulator"
- note added: "Button A"
- note added: "Button B"
- note added: "Button for State Machine"
- note added: "Buttons"
- note added: "CR2032 Battery Holder"
- note added: "Flip Flops"
- note added: "Input Power"
- note added: "Multiplexers take counter input and output states for 16 segment display"
- note added: "Negative Edge Triggered JK flip flop"
- note added: "On/Off Switch"
- note added: "Put a Schottky diode here with <300mV forward voltage at 400mA to use both battery and USB supplies"
- note added: "SR latch"
- note added: "Synchronous 3-Bit 0-5 Counter"
- note added: "USB-C Connector"
- note removed: "JK flip flop"
- note removed: "NOT gate"
- note removed: "SR flip flop"
- moved on the sheet: C1, DS1, R6, VR1
