File: Logic-PCB/Logic-PCB.kicad_sch (KiCad schematic)
At the start: 8 parts, among them Q1 MMBT2222, Q2 MMBT2907A-7-F, SW1 SW_Omron_B3FS, SW1 SW_Push

Commit message: stuff
Parts:
- removed Q2: MMBT2907A-7-F, SOT96P240X100-3N, symbol SamacSys_Parts:MMBT2907A-7-F
- removed R1 (x2): R, symbol Device:R
- removed SW1: SW_Omron_B3FS, symbol Switch:SW_Omron_B3FS
- added C1: 1u, symbol Device:C
- added C2: .01u, symbol Device:C
- added C3: .1u, symbol Device:C
- added D2, D3, D4, D5, D6: LED, symbol Device:LED
- added DS1: PSA08-11GWA, PSA0811GWA, symbol SamacSys_Parts:PSA08-11GWA
- added IC1, IC11, IC5, IC6: MC14027BDR2G, SOIC127P600X175-16N, symbol SamacSys_Parts:MC14027BDR2G
- added IC10: 74LVC1G08FW5-7, 74LVC1G08FW57, symbol SamacSys_Parts:74LVC1G08FW5-7
- added IC12, IC13, IC14, IC15, IC16, IC17, IC18, IC19, IC9: TMUX4051PWR, SOP65P640X120-16N, symbol SamacSys_Parts:TMUX4051PWR
- added IC2: LM555CMX_NOPB, SOIC127P600X175-8N, symbol SamacSys_Parts:LM555CMX_NOPB
- added IC3: NLV17SZ74USG, SOP50P310X90-8N, symbol SamacSys_Parts:NLV17SZ74USG
- added IC4: MC14043BDR2G, SOIC127P600X175-16N, symbol SamacSys_Parts:MC14043BDR2G
- added IC7: CD4082BM96, SOIC127P600X175-14N, symbol SamacSys_Parts:CD4082BM96
- added IC8: 74LVC1G32GV,125, SOT95P275X110-5N, symbol SamacSys_Parts:74LVC1G32GV,125
- added R1: R, symbol Device:R
- added R10, R12, R13, R14, R16, R8, R9: 10k, symbol Device:R
- added R11, R15, R3, R7: 51, symbol Device:R
- added R4, R5: 1k, symbol Device:R
- added R6: 220, symbol Device:R
- added SW2, SW3, SW4, SW5, SW6, SW7, SW8: SW_Push, symbol Switch:SW_Push
- added VR1: 3314J-2-105E, 3314J-1, symbol SamacSys_Parts:3314J-2-105E
Connections:
- net +5V: now also C3.1, IC2.4 (RESET), IC2.8 (+VCC), R4.1; no longer R2.1
- net GND: now also C1.2, C2.2, C3.2, D2.1 (K), D3.1 (K), D4.1 (K), D5.1 (K), D6.1 (K), IC1.4 (RA), IC1.7 (SA), IC1.8 (VSS), IC10.3 (GND), IC11.4 (RA), IC11.7 (SA), IC11.8 (VSS), IC12.1 (S4), IC12.12 (S3), IC12.13 (S0), IC12.14 (S1), IC12.2 (S6), IC12.4 (S7), IC12.5 (S5), IC12.6 (~{EN}), IC12.7 (VSS), IC12.8 (GND), IC13.1 (S4), IC13.12 (S3), IC13.14 (S1), IC13.2 (S6), IC13.4 (S7), IC13.5 (S5), IC13.6 (~{EN}), IC13.7 (VSS), IC13.8 (GND), IC14.6 (~{EN}), IC14.7 (VSS), IC14.8 (GND), IC15.6 (~{EN}), IC15.7 (VSS), IC15.8 (GND), IC16.6 (~{EN}), IC16.7 (VSS), IC16.8 (GND), IC17.6 (~{EN}), IC17.7 (VSS), IC17.8 (GND), IC18.6 (~{EN}), IC18.7 (VSS), IC18.8 (GND), IC19.6 (~{EN}), IC19.7 (VSS), IC19.8 (GND), IC2.1 (GND), IC3.4 (GND), IC4.8 (VSS), IC5.4 (RA), IC5.7 (SA), IC5.8 (VSS), IC6.12 (RB), IC6.4 (RA), IC6.7 (SA), IC6.8 (VSS), IC6.9 (SB), IC7.7 (VSS), IC8.3 (GND), IC9.15 (S2), IC9.2 (S6), IC9.4 (S7), IC9.5 (S5), IC9.6 (~{EN}), IC9.7 (VSS), IC9.8 (GND), R10.1, R12.1, R13.1, R14.1, R16.1, R8.1, R9.1
- net at SW1.2: now also R1.2
- new net: IC2.7 (DISCHARGE), R4.2, R5.2
- new net: IC4.3 (R0), R12.2, SW5.2
- new net: D2.2 (A), R3.1
- new net: IC1.1 (QA), R3.2
- new net: IC4.2 (Q0), R11.1
- new net: D5.2 (A), R11.2
- new net: IC1.6 (JA), R8.2, SW3.2
- new net: IC3.2 (D), R10.2, SW4.2
- new net: IC12.10 (A1), IC13.10 (A1), IC14.10 (A1), IC15.10 (A1), IC16.10 (A1), IC17.10 (A1), IC18.10 (A1), IC19.10 (A1), IC6.15 (QB), IC7.3 (C), IC9.10 (A1)
- new net: IC12.11 (A0), IC13.11 (A0), IC14.11 (A0), IC15.11 (A0), IC16.11 (A0), IC17.11 (A0), IC18.11 (A0), IC19.11 (A0), IC6.1 (QA), IC7.9 (E), IC9.11 (A0)
- new net: DS1.2 (K_M), DS1.6 (K_S), IC17.3 (D)
- new net: IC10.2 (B), IC11.1 (QA), IC12.9 (A2), IC13.9 (A2), IC14.9 (A2), IC15.9 (A2), IC16.9 (A2), IC17.9 (A2), IC18.9 (A2), IC19.9 (A2), IC7.11 (G), IC7.2 (D), IC9.9 (A2)
- new net: DS1.4 (K_H), DS1.8 (K_G), IC15.3 (D)
- new net: IC10.1 (A), IC6.2 (~{QA}), IC7.4 (B)
- new net: IC10.4 (Y), IC6.10 (JB), IC6.11 (KB)
- new net: IC3.5 (Q), R7.1
- new net: IC7.1 (J=A+B.C.D), IC8.1 (B)
- new net: IC7.13 (K=E.F.G.H), IC8.2 (A)
- new net: IC6.5 (KA), IC6.6 (JA), IC8.4 (Y)
- new net: IC4.4 (S0), R13.2, SW6.2
- new net: R5.1, VR1.2 (WIPER)
- new net: DS1.13 (K_D), IC13.3 (D)
- new net: DS1.16 (K_C), IC12.3 (D)
- new net: DS1.1 (K_A), DS1.18 (K_B), IC9.3 (D)
- new net: DS1.10 (K_E), DS1.15 (K_P), DS1.9 (K_F), IC14.3 (D)
- new net: DS1.14 (K_R), DS1.3 (K_K), IC16.3 (D)
- new net: DS1.17 (K_N), DS1.7 (K_T), IC18.3 (D)
- new net: DS1.5 (K_U), IC19.3 (D)
- new net: D3.2 (A), R6.2
- new net: IC6.14 (~{QB}), IC7.10 (F)
- new net: D6.2 (A), R15.1
- new net: D4.2 (A), R7.2
- new net: IC5.1 (QA), R15.2
- new net: IC5.5 (KA), IC5.6 (JA), R16.2, SW7.2
- new net: IC1.5 (KA), R9.2, SW2.2
- new net: C2.1, IC2.5 (CONTROL_VOLTAGE)
- new net: C1.1, IC2.2 (TRIGGER), IC2.6 (THRESHOLD), VR1.3 (CW)
- new net +3V0: IC1.16 (VDD), IC10.6 (VCC), IC11.5 (KA), IC11.6 (JA), IC12.15 (S2), IC12.16 (VDD), IC13.13 (S0), IC13.15 (S2), IC13.16 (VDD), IC14.1 (S4), IC14.13 (S0), IC14.14 (S1), IC14.16 (VDD), IC15.1 (S4), IC15.13 (S0), IC15.14 (S1), IC15.15 (S2), IC15.16 (VDD), IC16.15 (S2), IC16.16 (VDD), IC16.5 (S5), IC17.12 (S3), IC17.16 (VDD), IC18.16 (VDD), IC18.5 (S5), IC19.1 (S4), IC19.14 (S1), IC19.16 (VDD), IC3.6 (~{CLR}), IC3.7 (~{PR}), IC3.8 (VCC), IC4.16 (VDD), IC5.16 (VDD), IC6.16 (VDD), IC7.14 (VDD), IC8.5 (VCC), IC9.1 (S4), IC9.12 (S3), IC9.13 (S0), IC9.14 (S1), IC9.16 (VDD), R1.1, R2.1, SW2.1, SW3.1, SW4.1, SW5.1, SW6.1, SW7.1, SW8.1
- new net Button: IC11.3 (CA), IC6.13 (CB), IC6.3 (CA), R14.2, SW8.2
- new net CLK: IC1.3 (CA), IC2.3 (OUTPUT), IC3.1 (CP), IC4.5 (E), IC5.3 (CA), R6.1
Other:
- note added: "AND gate"
- note added: "Adjustable Timer"
- note added: "D flip flop"
- note added: "JK flip flop"
- note added: "NOT gate"
- note added: "OR gate"
- note added: "SR flip flop"
- note added: "T flip flop"
- note added: "To reduce noise on rising edge"
- note added: "To stabilize power supply (put close as possible to chip)"

Commit message: gates
Parts:
- added D1, D4 (x6): LED, LED_SMD:LED_0402_1005Metric, symbol Device:LED
- added IC1: 74AUP1T87GWH, SOT65P212X110-5N, symbol SamacSys_Parts:74AUP1T87GWH
- added Q1 (x8): MMBT2222, SamacSys_Parts:SOT95P240X114-3N, symbol SamacSys_Parts:MMBT2222
- added Q1, Q10, Q11, Q8, Q9: MMBT2907A-7-F, SOT96P240X100-3N, symbol SamacSys_Parts:MMBT2907A-7-F
- added R1, R18, R19, R20, R21, R23, R24, R25, R26, R3, R4, R5, R6: 5.6k, Resistor_SMD:R_0402_1005Metric, symbol Device:R
- added R10 (x13): 10k, Resistor_SMD:R_0402_1005Metric, symbol Device:R
- added R17, R2, R22, R27, R32, R33, R7: 51, Resistor_SMD:R_0402_1005Metric, symbol Device:R
- added SW4 (x13): SW_Push, symbol Switch:SW_Push
- added U1: 74AHC1G86W5-7, SOT95P285X130-5N, symbol SamacSys_Parts:74AHC1G86W5-7
Connections:
- net GND is gone; now on net +3V0: C1.2, C2.2, C3.2, D1.1 (K), D2.1 (K), D3.1 (K), D4.1 (K), D5.1 (K), D6.1 (K), IC1.4 (RA), IC1.7 (SA), IC1.8 (VSS), IC10.3 (GND), IC11.4 (RA), IC11.7 (SA), IC11.8 (VSS), IC12.1 (S4), IC12.12 (S3), IC12.13 (S0), IC12.14 (S1), IC12.2 (S6), IC12.4 (S7), IC12.5 (S5), IC12.6 (~{EN}), IC12.7 (VSS), IC12.8 (GND), IC13.1 (S4), IC13.12 (S3), IC13.14 (S1), IC13.2 (S6), IC13.4 (S7), IC13.5 (S5), IC13.6 (~{EN}), IC13.7 (VSS), IC13.8 (GND), IC14.6 (~{EN}), IC14.7 (VSS), IC14.8 (GND), IC15.6 (~{EN}), IC15.7 (VSS), IC15.8 (GND), IC16.6 (~{EN}), IC16.7 (VSS), IC16.8 (GND), IC17.6 (~{EN}), IC17.7 (VSS), IC17.8 (GND), IC18.6 (~{EN}), IC18.7 (VSS), IC18.8 (GND), IC19.6 (~{EN}), IC19.7 (VSS), IC19.8 (GND), IC2.1 (GND), IC3.4 (GND), IC4.8 (VSS), IC5.4 (RA), IC5.7 (SA), IC5.8 (VSS), IC6.12 (RB), IC6.4 (RA), IC6.7 (SA), IC6.8 (VSS), IC6.9 (SB), IC7.7 (VSS), IC8.3 (GND), IC9.15 (S2), IC9.2 (S6), IC9.4 (S7), IC9.5 (S5), IC9.6 (~{EN}), IC9.7 (VSS), IC9.8 (GND), Q1.2, R10.1, R12.1, R13.1, R14.1, R16.1, R8.1, R9.1
- net +3V0: now also D4.1 (K), D4.1 (K), D4.1 (K), D4.1 (K), D4.1 (K), D4.1 (K), IC1.3 (GND), IC1.5 (VCC), Q1.2, Q1.2, Q1.2, Q1.3, Q1.3, Q1.3, Q1.3, Q10.2, Q8.2, Q9.2, R10.1, R10.1, R10.1, R10.1, R10.1, R10.1, R10.1, R10.1, R10.1, R10.1, R10.1, R10.1, R10.1, R2.1, SW4.1, SW4.1, SW4.1, SW4.1, SW4.1, SW4.1, SW4.1, SW4.1, SW4.1, SW4.1, SW4.1, SW4.1, SW4.1, U1.3 (GND), U1.5 (VCC)
- new net: R1.1, R10.2, SW4.2
- new net: R10.2, R5.1, R6.1, SW4.2
- new net: Q1.1, R6.2
- new net: D4.2 (A), R27.1
- new net: D4.2 (A), R32.2
- new net: R10.2, SW4.2, U1.1 (A)
- new net: Q10.1, R3.1
- new net: R10.2, R3.2, R4.1, SW4.2
- new net: D1.1 (K), Q1.2
- new net: D1.2 (A), R2.2
- new net: R10.2, R19.1, SW4.2
- new net: R10.2, R18.1, SW4.2
- new net: Q1.1, R18.2
- new net: Q1.2, Q1.3 (x2)
- new net: R10.2, R23.1, R26.1, SW4.2
- new net: Q8.1, R26.2
- new net: IC1.4 (Y), R33.1
- new net: D4.2 (A), R33.2
- new net: R10.2, R21.1, SW4.2
- new net: IC1.2 (A), R10.2, SW4.2
- new net: IC1.1 (B), R10.2, SW4.2
- new net: Q1.1, R20.2
- new net: Q1.2, Q1.2, R22.2
- new net: R10.2, R20.1, SW4.2
- new net: D4.2 (A), R7.1
- new net: Q1.3, Q1.3, Q11.3, R7.2
- new net: Q1.1, R21.2
- new net: R10.2, R24.1, R25.1, SW4.2
- new net: Q9.1, R25.2
- new net: D4.2 (A), R22.1
- new net: Q10.3, Q11.2
- new net: Q11.1, R5.2
- new net: Q1.1, R23.2
- new net: Q1.1, R19.2
- new net: Q1.3, Q8.3, Q9.3, R27.2
- new net: Q1.1, R24.2
- new net: R10.2, SW4.2, U1.2 (B)
- new net: D4.2 (A), R17.1
- new net: Q1.2, R17.2
- new net: R32.1, U1.4 (Y)
- new net: Q1.1, R4.2
- new net: Q1.1, R1.2
Other:
- note added: "AND Gate"
- note added: "NAND Gate"
- note added: "NOR Gate"
- note added: "NOT Gate"
- note added: "OR Gate"
- note added: "XNOR Gate"
- note added: "XOR Gate"

Commit message: Update Logic-PCB.kicad_sch
Parts:
- removed D4 (x6): LED, LED_SMD:LED_0402_1005Metric, symbol Device:LED
- removed Q1 (x8): MMBT2222, SamacSys_Parts:SOT95P240X114-3N, symbol SamacSys_Parts:MMBT2222
- removed R10 (x13): 10k, Resistor_SMD:R_0402_1005Metric, symbol Device:R
- removed SW4 (x13): SW_Push, symbol Switch:SW_Push
- added D4 (x6): LED, LED_SMD:LED_0402_1005Metric, symbol Device:LED
- added Q1 (x8): MMBT2222, SamacSys_Parts:SOT95P240X114-3N, symbol SamacSys_Parts:MMBT2222
- added R10 (x13): 10k, Resistor_SMD:R_0402_1005Metric, symbol Device:R
- added SW4 (x13): SW_Push, SamacSys_Parts:EVPASAC1A, symbol Switch:SW_Push
Connections:
- net +3V0: now also D4.1 (K), D4.1 (K), D4.1 (K), D4.1 (K), D4.1 (K), D4.1 (K), Q1.2, Q1.2, Q1.2, Q1.3, Q1.3, Q1.3, R10.1, R10.1, R10.1, R10.1, R10.1, R10.1, R10.1, R10.1, R10.1, R10.1, R10.1, R10.1, R10.1, SW4.1, SW4.1, SW4.1, SW4.1, SW4.1, SW4.1, SW4.1, SW4.1, SW4.1, SW4.1, SW4.1, SW4.1, SW4.1
- net at R1.1: now also R10.2, SW4.2
- net at R5.1, R6.1: now also R10.2, SW4.2
- net at R6.2: now also Q1.1
- net at R27.1: now also D4.2 (A)
- net at R32.2: now also D4.2 (A)
- net at U1.1 (A): now also R10.2, SW4.2
- net at R3.2, R4.1: now also R10.2, SW4.2
- net at R19.1: now also R10.2, SW4.2
- net at R18.1: now also R10.2, SW4.2
- net at R18.2: now also Q1.1
- net at R23.1, R26.1: now also R10.2, SW4.2
- net at R33.2: now also D4.2 (A)
- net at R21.1: now also R10.2, SW4.2
- net at IC1.2 (A): now also R10.2, SW4.2
- net at IC1.1 (B): now also R10.2, SW4.2
- net at R20.2: now also Q1.1
- net at R22.2: now also Q1.2, Q1.2
- net at R20.1: now also R10.2, SW4.2
- net at R7.1: now also D4.2 (A)
- net at Q11.3, R7.2: now also Q1.3, Q1.3
- net at R21.2: now also Q1.1
- net at R24.1, R25.1: now also R10.2, SW4.2
- net at R22.1: now also D4.2 (A)
- net at R23.2: now also Q1.1
- net at R19.2: now also Q1.1
- net at Q8.3, Q9.3, R27.2: now also Q1.3
- net at R24.2: now also Q1.1
- net at U1.2 (B): now also R10.2, SW4.2
- net at R17.1: now also D4.2 (A)
- net at R17.2: now also Q1.2
- net at R4.2: now also Q1.1
- new net: Q1.2, Q1.3 (x2)

Commit message: Gates
Parts:
- removed D4 (x6): LED, LED_SMD:LED_0402_1005Metric, symbol Device:LED
- removed Q1 (x8): MMBT2222, SamacSys_Parts:SOT95P240X114-3N, symbol SamacSys_Parts:MMBT2222
- removed Q8: MMBT2907A-7-F, SOT96P240X100-3N, symbol SamacSys_Parts:MMBT2907A-7-F
- removed R1, R21, R23, R24, R25, R26: 5.6k, Resistor_SMD:R_0402_1005Metric, symbol Device:R
- removed R10 (x13): 10k, Resistor_SMD:R_0402_1005Metric, symbol Device:R
- removed R2, R22, R27, R32, R33: 51, Resistor_SMD:R_0402_1005Metric, symbol Device:R
- removed SW4 (x13): SW_Push, SamacSys_Parts:EVPASAC1A, symbol Switch:SW_Push
- added D4 (x6): LED, LED_SMD:LED_0402_1005Metric, symbol Device:LED
- added Q1 (x8): MMBT2222, SamacSys_Parts:SOT95P240X114-3N, symbol SamacSys_Parts:MMBT2222
- added Q2: MMBT2907A-7-F, SOT96P240X100-3N, symbol SamacSys_Parts:MMBT2907A-7-F
- added R1 (x2), R14, R15, R16, R2, R8: 5.6k, Resistor_SMD:R_0402_1005Metric, symbol Device:R
- added R10, R11, R2, R9: 51, Resistor_SMD:R_0402_1005Metric, symbol Device:R
- R17, R7: value 51 -> 5.6k
- R18, R19, R20: value 5.6k -> 51
Connections:
- net +3V0: now also Q1.2, Q9.3, D4.1 (K), D4.1 (K), D4.1 (K), D4.1 (K), D4.1 (K), D4.1 (K), Q1.2, Q1.2, Q1.2, Q1.3, Q1.3, Q1.3, Q2.2, R2.1; no longer Q1.3, Q9.2
- net at IC1.4 (Y): now also R20.1
- net Button B: now reaches R17.1
- net Button B: now also IC1.2 (A), R3.1, R4.1, R6.1, U1.2 (B), R15.1, R8.1
- net at R17.2: now also Q11.1
- net Button A: now reaches R5.1
- net Button A: now also IC1.1 (B), R7.1, U1.1 (A), R1.1, R1.1, R14.2, R16.1, R2.1; no longer R6.1
- net at R5.2: now also Q1.1; no longer Q11.1
- net at R18.1: now also U1.4 (Y)
- net at R18.2: now also D4.2 (A)
- net at R3.2: now also Q2.1; no longer R4.1
- net at Q9.1: now also R1.2
- net at R19.1: now also D4.2 (A)
- net at R6.2: now also Q1.1
- net at R7.2: now also Q1.1; no longer Q11.3
- net at Q10.1: now also R14.1; no longer R3.1
- net at Q1.1: now also R1.2
- net at R20.2: now also D4.2 (A)
- net at D1.1 (K): now also Q9.2; no longer Q1.2
- net at D1.2 (A): now also R2.2
- net at R19.2: now also Q11.3, Q1.3, Q1.3
- net at R4.2: now also Q1.1
- new net: Q1.2, Q1.3 (x2)
- new net: Q1.3, Q1.3, Q2.3, R11.2
- new net: D4.2 (A), R11.1
- new net: D4.2 (A), R10.1
- new net: Q1.1, R15.2
- new net: Q1.1, R2.2
- new net: Q1.2, Q1.2, R10.2
- new net: D4.2 (A), R9.1
- new net: Q1.1, R8.2
- new net: Q1.2, R9.2
- new net: Q1.1, R16.2
