File: Logic-PCB/Logic-PCB.kicad_sch (KiCad schematic)
At the start: 118 parts, among them IC1 74AUP1T87GWH, IC1 74LVC1G74DC-Q100H, IC10 SN74LVC1G11MDCKREP, IC11 SN74LVC1G97QDBVRQ1, IC12 SN74LVC1G97QDBVRQ1, IC13 TMUX1208QRSVRQ1, IC14 TMUX1208QRSVRQ1, IC15 TMUX1208QRSVRQ1, IC16 TMUX1208QRSVRQ1, IC17 TMUX1208QRSVRQ1, IC18 TMUX1208QRSVRQ1, IC19 TMUX1208QRSVRQ1, IC2 74HC73D,653, IC20 TMUX1208QRSVRQ1, IC21 TMUX1208QRSVRQ1, IC3 TLC555QDRQ1, IC4 SN74LVC1G02DBVR, IC5 SN74LVC1G02DBVR, IC6 NCV4274AST33T3G, IC7 74HC73D,653, IC8 74HC73D,653, IC9 SN74LVC1G11MDCKREP, J1 CX70M-24P1, Q1 MMBT2222, Q1 MMBT2907A-7-F, Q10 MMBT2907A-7-F, Q11 MMBT2907A-7-F, Q2 MMBT2907A-7-F, Q9 MMBT2907A-7-F, SW1 SW_Push, SW2 SW_Push, SW3 SW_Push, U1 74AHC1G86W5-7, U1 BAT-HLD-001-TR

Commit message: Gates (R change)
Parts:
- R10, R11, R18, R19, R2, R20, R9: value 51 -> 100
Changed lines of the file:
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@@
   (junction (at 96.52 54.61) (diameter 0) (color 0 0 0 0)
   )
-  (junction (at 103.378 350.012) (diameter 0) (color 0 0 0 0)
-  )
   (junction (at 97.79 173.99) (diameter 0) (color 0 0 0 0)
   )
@@
   (junction (at 378.46 243.84) (diameter 0) (color 0 0 0 0)
   )
+  (junction (at 103.378 350.012) (diameter 0) (color 0 0 0 0)
+  )
   (junction (at 57.15 106.68) (diameter 0) (color 0 0 0 0)
   )
@@
   (junction (at 176.53 360.934) (diameter 0) (color 0 0 0 0)
   )
-  (junction (at 103.378 349.758) (diameter 0) (color 0 0 0 0)
-  )
   (junction (at 469.9 215.9) (diameter 0) (color 0 0 0 0)
   )
@@
     (stroke (width 0) (type default))
   )
+  (wire (pts (xy 103.378 350.012) (xy 112.776 350.012))
+    (stroke (width 0) (type default))
+  )
   (wire (pts (xy 590.55 199.39) (xy 590.55 195.58))
     (stroke (width 0) (type default))
@@
     (stroke (width 0) (type default))
   )
-  (wire (pts (xy 103.378 350.012) (xy 103.378 351.282))
+  (wire (pts (xy 469.9 57.15) (xy 469.9 88.9))
     (stroke (width 0) (type default))
   )
-  (wire (pts (xy 469.9 57.15) (xy 469.9 88.9))
+  (wire (pts (xy 103.378 350.012) (xy 103.378 351.282))
     (stroke (width 0) (type default))
   )
@@
     (stroke (width 0) (type default))
   )
-  (wire (pts (xy 112.776 349.758) (xy 112.776 356.108))
+  (wire (pts (xy 112.776 350.012) (xy 112.776 356.108))
     (stroke (width 0) (type default))
   )
@@
     (stroke (width 0) (type default))
   )
-  (wire (pts (xy 88.138 350.012) (xy 103.378 350.012))
+  (wire (pts (xy 378.46 219.71) (xy 378.46 236.22))
     (stroke (width 0) (type default))
   )
-  (wire (pts (xy 378.46 219.71) (xy 378.46 236.22))
+  (wire (pts (xy 103.378 348.742) (xy 103.378 350.012))
     (stroke (width 0) (type default))
   )
@@
     (stroke (width 0) (type default))
   )
-  (wire (pts (xy 103.378 349.758) (xy 103.378 350.012))
-    (stroke (width 0) (type default))
-  )
   (wire (pts (xy 435.61 46.99) (xy 435.61 54.61))
     (stroke (width 0) (type default))
@@
     (stroke (width 0) (type default))
   )
-  (wire (pts (xy 103.378 349.758) (xy 112.776 349.758))
+  (wire (pts (xy 88.138 350.012) (xy 103.378 350.012))
     (stroke (width 0) (type default))
   )
@@
     (stroke (width 0) (type default))
   )
-  (wire (pts (xy 103.378 348.742) (xy 103.378 349.758))
-    (stroke (width 0) (type default))
-  )
   (wire (pts (xy 467.36 118.11) (xy 467.36 149.86))
     (stroke (width 0) (type default))
@@
       (effects (font (size 1.27 1.27)) (justify left))
     )
-    (property "Value" "51" (at 196.342 256.54 0)
+    (property "Value" "100" (at 196.342 256.54 0)
       (effects (font (size 1.27 1.27)) (justify left))
     )
@@
       (effects (font (size 1.27 1.27)) (justify right))
     )
-    (property "Value" "51" (at 180.848 351.282 0)
+    (property "Value" "100" (at 180.848 351.282 0)
       (effects (font (size 1.27 1.27)) (justify right))
     )
@@
       (effects (font (size 1.27 1.27)) (justify left))
     )
-    (property "Value" "51" (at 142.748 257.302 0)
+    (property "Value" "100" (at 142.748 257.302 0)
       (effects (font (size 1.27 1.27)) (justify left))
     )
@@
       (effects (font (size 1.27 1.27)))
     )
-    (property "Value" "51" (at 189.484 297.688 90)
+    (property "Value" "100" (at 189.484 297.688 90)
       (effects (font (size 1.27 1.27)))
     )
@@
       (effects (font (size 1.27 1.27)) (justify right))
     )
-    (property "Value" "51" (at 115.316 361.188 0)
+    (property "Value" "100" (at 115.316 361.188 0)
       (effects (font (size 1.27 1.27)) (justify right))
     )
@@
       (effects (font (size 1.27 1.27)))
     )
-    (property "Value" "51" (at 77.47 279.146 90)
+    (property "Value" "100" (at 77.47 279.146 90)
       (effects (font (size 1.27 1.27)))
     )
@@
       (effects (font (size 1.27 1.27)))
     )
-    (property "Value" "51" (at 76.708 326.136 90)
+    (property "Value" "100" (at 76.708 326.136 90)
       (effects (font (size 1.27 1.27)))
     )

Commit message: Decoupling Caps
Parts:
- added C4 (x21): .1u, Capacitor_SMD:C_01005_0402Metric, symbol Device:C
Connections:
- net +3V0: now also C4.1, C4.1, C4.1, C4.1, C4.1, C4.1, C4.1, C4.1, C4.1, C4.1, C4.1, C4.1, C4.1, C4.1, C4.1, C4.1, C4.1, C4.1, C4.1, C4.1, C4.1, C4.2, C4.2, C4.2, C4.2, C4.2, C4.2, C4.2, C4.2, C4.2, C4.2, C4.2, C4.2, C4.2, C4.2, C4.2, C4.2, C4.2, C4.2, C4.2, C4.2, C4.2
Other:
- note added: "555 Timer"
- note added: "8 to 1 Mux"
- note added: "Adjustable Clock Generator"
- note added: "Decoupling cap to stabilize power supply (put close as possible to chip)"
- note added: "Multiplexers take counter input and output states for 16 segment display, which cycles through the letters GENTEX"
- note added: "NOR"
- note added: "Potentiometer to change frequency of clock pulse"
- note added: "Put a Schottky diode here with <300mV forward voltage at 300mA to use both battery and USB supplies"
- note added: "Synchronous 3-Bit 0 to 5 Counter (also displays function of T flip flops with LEDs)"
- note removed: "Adjustable Timer"
- note removed: "Multiplexers take counter input and output states for 16 segment display"
- note removed: "Put a Schottky diode here with <300mV forward voltage at 400mA to use both battery and USB supplies"
- note removed: "Synchronous 3-Bit 0-5 Counter"
- note removed: "To stabilize power supply (put close as possible to chip)"
- company: (none) -> Gentex Corporation
- title: (none) -> Quick Turn Promotional PCB
- moved on the sheet: C1, C2, C3, C4, C5, D1, D10, D11, D12, D2, D3, D4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

Commit message: Gates
Connections:
- net +3V0: no longer C1.2, C2.2, C3.2, C4.1, C4.2, C4.2, C4.2, C4.2, C4.2, C4.2, C4.2, C4.2, C4.2, C4.2, C4.2, C4.2, C4.2, C4.2, C4.2, C4.2, C4.2, C4.2, C4.2, C4.2, C4.2, C5.2, D1.1 (K), D10.1 (K), D11.1 (K), D12.1 (K), D2.1 (K), D3.1 (K), D4.1 (K), D4.1 (K), D4.1 (K), D4.1 (K), D4.1 (K), D4.1 (K), D4.1 (K), D5.1 (K), D7.1 (K), D8.1 (K), D9.1 (K), DS1.11 (COM_A), DS1.12 (K_DP), IC1.3 (GND), IC1.4 (GND), IC10.2 (GND), IC11.2 (GND), IC12.1 (IN1), IC12.2 (GND), IC13.12 (GND), IC13.4 (S3), IC13.7 (S8), IC13.8 (S7), IC13.9 (S6), IC14.10 (S5), IC14.12 (GND), IC14.2 (S1), IC14.3 (S2), IC14.5 (S4), IC14.7 (S8), IC14.8 (S7), IC14.9 (S6), IC15.10 (S5), IC15.12 (GND), IC15.3 (S2), IC15.5 (S4), IC15.7 (S8), IC15.8 (S7), IC15.9 (S6), IC16.12 (GND), IC16.4 (S3), IC16.5 (S4), IC16.7 (S8), IC16.8 (S7), IC16.9 (S6), IC17.12 (GND), IC17.5 (S4), IC17.7 (S8), IC17.8 (S7), IC17.9 (S6), IC18.10 (S5), IC18.12 (GND), IC18.2 (S1), IC18.3 (S2), IC18.5 (S4), IC18.7 (S8), IC18.8 (S7), IC19.10 (S5), IC19.12 (GND), IC19.2 (S1), IC19.3 (S2), IC19.4 (S3), IC19.7 (S8), IC19.8 (S7), IC19.9 (S6), IC2.11 (GND), IC20.10 (S5), IC20.12 (GND), IC20.2 (S1), IC20.3 (S2), IC20.4 (S3), IC20.5 (S4), IC20.7 (S8), IC20.8 (S7), IC21.12 (GND), IC21.2 (S1), IC21.4 (S3), IC21.5 (S4), IC21.7 (S8), IC21.8 (S7), IC21.9 (S6), IC3.1 (GND), IC4.3 (GND), IC5.3 (GND), IC6.2 (GROUND_1), IC6.4 (GROUND_2), IC7.11 (GND), IC8.11 (GND), IC9.2 (GND), J1.A1 (GND_1), J1.A12 (GND_2), J1.B1 (GND_3), J1.B12 (GND_4), Q1.2, Q1.2, Q1.2, Q9.3, R1.1, R13.1, R14.1, R15.1, R2.1, R4.1, R7.1, R8.1, S1.3 (COM_1), S1.7 (COM_2), U1.3, U1.3 (GND)
- new net GND: C1.2, C2.2, C3.2, C4.1, C4.2, C4.2, C4.2, C4.2, C4.2, C4.2, C4.2, C4.2, C4.2, C4.2, C4.2, C4.2, C4.2, C4.2, C4.2, C4.2, C4.2, C4.2, C4.2, C4.2, C4.2, C5.2, D1.1 (K), D10.1 (K), D11.1 (K), D12.1 (K), D2.1 (K), D3.1 (K), D4.1 (K), D4.1 (K), D4.1 (K), D4.1 (K), D4.1 (K), D4.1 (K), D4.1 (K), D5.1 (K), D7.1 (K), D8.1 (K), D9.1 (K), DS1.11 (COM_A), DS1.12 (K_DP), IC1.3 (GND), IC1.4 (GND), IC10.2 (GND), IC11.2 (GND), IC12.1 (IN1), IC12.2 (GND), IC13.12 (GND), IC13.4 (S3), IC13.7 (S8), IC13.8 (S7), IC13.9 (S6), IC14.10 (S5), IC14.12 (GND), IC14.2 (S1), IC14.3 (S2), IC14.5 (S4), IC14.7 (S8), IC14.8 (S7), IC14.9 (S6), IC15.10 (S5), IC15.12 (GND), IC15.3 (S2), IC15.5 (S4), IC15.7 (S8), IC15.8 (S7), IC15.9 (S6), IC16.12 (GND), IC16.4 (S3), IC16.5 (S4), IC16.7 (S8), IC16.8 (S7), IC16.9 (S6), IC17.12 (GND), IC17.5 (S4), IC17.7 (S8), IC17.8 (S7), IC17.9 (S6), IC18.10 (S5), IC18.12 (GND), IC18.2 (S1), IC18.3 (S2), IC18.5 (S4), IC18.7 (S8), IC18.8 (S7), IC19.10 (S5), IC19.12 (GND), IC19.2 (S1), IC19.3 (S2), IC19.4 (S3), IC19.7 (S8), IC19.8 (S7), IC19.9 (S6), IC2.11 (GND), IC20.10 (S5), IC20.12 (GND), IC20.2 (S1), IC20.3 (S2), IC20.4 (S3), IC20.5 (S4), IC20.7 (S8), IC20.8 (S7), IC21.12 (GND), IC21.2 (S1), IC21.4 (S3), IC21.5 (S4), IC21.7 (S8), IC21.8 (S7), IC21.9 (S6), IC3.1 (GND), IC4.3 (GND), IC5.3 (GND), IC6.2 (GROUND_1), IC6.4 (GROUND_2), IC7.11 (GND), IC8.11 (GND), IC9.2 (GND), J1.A1 (GND_1), J1.A12 (GND_2), J1.B1 (GND_3), J1.B12 (GND_4), Q1.2, Q1.2, Q1.2, Q9.3, R1.1, R13.1, R14.1, R15.1, R2.1, R4.1, R7.1, R8.1, S1.3 (COM_1), S1.7 (COM_2), U1.3, U1.3 (GND)
Other:
- moved on the sheet: C4, D4, Q1, Q2, R1, R11, R18, R19, R2, R20, R3, R4

Commit message: Removing pulldown resistors
Parts:
- removed R1, R2, R4, R7, R8: 10k, Resistor_SMD:R_0402_1005Metric, symbol Device:R

Commit message: updates from meeting
Parts:
- removed IC12: SN74LVC1G97QDBVRQ1, SamacSys_Parts:SOT95P280X145-6N, symbol SamacSys_Parts:SN74LVC1G97QDBVRQ1
- removed IC6: NCV4274AST33T3G, SamacSys_Parts:SOT230P700X175-4N, symbol SamacSys_Parts:NCV4274AST33T3G
- removed R15: 10k, Resistor_SMD:R_0402_1005Metric, symbol Device:R
- removed SW3: SW_Push, SamacSys_Parts:SKPMBHE010, symbol Switch:SW_Push
- added C5 (x3): .1u, Capacitor_SMD:C_01005_0402Metric, symbol Device:C
- added C5 (x2): 1u, Capacitor_SMD:C_01005_0402Metric, symbol Device:C
- added D6: LSM115JE3_TR13, SamacSys_Parts:DIOM5436X330N, symbol SamacSys_Parts:LSM115JE3_TR13
- added IC23: NCV4274CDT33RKG, NCV4274CDT33RKG, symbol SamacSys_Parts:NCV4274CDT33RKG
- added R5 (x2): 5.1k, Resistor_SMD:R_0402_1005Metric, symbol Device:R
- added U3: NC7S08M5X, SOT95P280X145-5N, symbol SamacSys_Parts:NC7S08M5X
Connections:
- net Button is gone; now on net CLK: IC7.1 (1~{CP}), IC8.1 (1~{CP}), IC8.5 (2~{CP})
- net +3V0: now also U3.5 (VCC)
- net +5V: now also IC23.1 (INPUT)
- net 3V before switch: now also D6.1; no longer C5.1
- net Button A: now also C5.1, C5.1
- net Button B: now also C5.1, C5.1
- net GND: now also C5.2, C5.2, C5.2, C5.2, C5.2, IC23.2 (GROUND), R5.1, R5.1, U3.3 (GND)
- net at J1.A5 (CC1): now also R5.2
- net at J1.B5 (CC2): now also R5.2
- net at IC8.10 (2K), IC8.7 (2J), R17.2: now also U3.4 (Y)
- net at IC10.6 (C), IC8.13 (1~{Q}): now also U3.1 (A)
- net at IC10.3 (B), IC13.13 (A2), IC14.13 (A2)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: now also U3.2 (B)
- new net: C5.1, C5.1, D6.2, IC23.3 (OUTPUT)
- no-connect marks 43 -> 41
Other:
- note added: "C"
- note added: "RA"
- note added: "RB"
- note removed: "Button for State Machine"
- moved on the sheet: C1, C2, C3, C4, C5, D10, D11, D12, D3, D7, D8, D9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

Commit message: CMOS
Parts:
- removed C4 (x21), C5 (x3): .1u, Capacitor_SMD:C_01005_0402Metric, symbol Device:C
- removed C4: 100n, Capacitor_SMD:C_01005_0402Metric, symbol Device:C
- removed C5 (x2): 1u, Capacitor_SMD:C_01005_0402Metric, symbol Device:C
- removed C5: 10u, Capacitor_SMD:C_01005_0402Metric, symbol Device:C
- removed D1 (x2), D10, D4 (x7), D9: LED, LED_SMD:LED_0402_1005Metric, symbol Device:LED
- removed D6 (x2): LSM115JE3_TR13, SamacSys_Parts:DIOM5436X330N, symbol SamacSys_Parts:LSM115JE3_TR13
- removed IC1: 74AUP1T87GWH, SOT65P212X110-5N, symbol SamacSys_Parts:74AUP1T87GWH
- removed IC11: SN74LVC1G97QDBVRQ1, SamacSys_Parts:SOT95P280X145-6N, symbol SamacSys_Parts:SN74LVC1G97QDBVRQ1
- removed IC23: NCV4274CDT33RKG, NCV4274CDT33RKG, symbol SamacSys_Parts:NCV4274CDT33RKG
- removed IC3: TLC555QDRQ1, SamacSys_Parts:SOIC127P600X175-8N, symbol SamacSys_Parts:TLC555QDRQ1
- removed IC5: SN74LVC1G02DBVR, SamacSys_Parts:SOT95P280X145-5N, symbol SamacSys_Parts:SN74LVC1G02DBVR
- removed IC8: 74HC73D,653, SamacSys_Parts:SOIC127P600X175-14N, symbol SamacSys_Parts:74HC73D,653
- removed IC9: SN74LVC1G11MDCKREP, SamacSys_Parts:SOP65P210X110-6N, symbol SamacSys_Parts:SN74LVC1G11MDCKREP
- removed Q1 (x8): MMBT2222, SamacSys_Parts:SOT95P240X114-3N, symbol SamacSys_Parts:MMBT2222
- removed Q1, Q11, Q2: MMBT2907A-7-F, SOT96P240X100-3N, symbol SamacSys_Parts:MMBT2907A-7-F
- removed R1 (x2), R14, R16, R17, R2, R3, R5, R6: 5.6k, Resistor_SMD:R_0402_1005Metric, symbol Device:R
- removed R10 (x2), R11 (x2), R16, R17, R18 (x2), R19 (x2), R2, R20 (x2), R3, R5, R6, R9: 100, Resistor_SMD:R_0402_1005Metric, symbol Device:R
- removed R14: 10k, Resistor_SMD:R_0402_1005Metric, symbol Device:R
- removed R5 (x2): 5.1k, Resistor_SMD:R_0402_1005Metric, symbol Device:R
- removed R9: 1k, Resistor_SMD:R_0402_1005Metric, symbol Device:R
- removed U1: BAT-HLD-001-TR, SamacSys_Parts:BATHLD001TR, symbol SamacSys_Parts:BAT-HLD-001-TR
- added C10, C11, C15: 1u, Capacitor_SMD:C_01005_0402Metric, symbol Device:C
- added C12, C13, C14, C16, C18, C19, C20, C21, C22, C23, C24, C25, C26, C27, C28, C29, C30, C31, C4, C5, C8, C9: .1u, Capacitor_SMD:C_01005_0402Metric, symbol Device:C
- added C17: .01u, Capacitor_SMD:C_01005_0402Metric, symbol Device:C
- added C6: 10u, Capacitor_SMD:C_01005_0402Metric, symbol Device:C
- added C7: 100n, Capacitor_SMD:C_01005_0402Metric, symbol Device:C
- added D1, D13, D14, D15, D16, D17, D18, D19, D20, D4, D6: LED, LED_SMD:LED_0402_1005Metric, symbol Device:LED
- added D10, D9: LSM115JE3_TR13, SamacSys_Parts:DIOM5436X330N, symbol SamacSys_Parts:LSM115JE3_TR13
- added IC11: SN74LVC1G11MDCKREP, SamacSys_Parts:SOP65P210X110-6N, symbol SamacSys_Parts:SN74LVC1G11MDCKREP
- added IC12: SN74LVC1G97QDBVRQ1, SamacSys_Parts:SOT95P280X145-6N, symbol SamacSys_Parts:SN74LVC1G97QDBVRQ1
- added IC3: SN74LVC1G02DBVR, SamacSys_Parts:SOT95P280X145-5N, symbol SamacSys_Parts:SN74LVC1G02DBVR
- added IC5: 74AUP1T87GWH, SOT65P212X110-5N, symbol SamacSys_Parts:74AUP1T87GWH
- added IC6: NCV4274CDT33RKG, NCV4274CDT33RKG, symbol SamacSys_Parts:NCV4274CDT33RKG
- added IC8: TLC555QDRQ1, SamacSys_Parts:SOIC127P600X175-8N, symbol SamacSys_Parts:TLC555QDRQ1
- added IC9: 74HC73D,653, SamacSys_Parts:SOIC127P600X175-14N, symbol SamacSys_Parts:74HC73D,653
- added Q1, Q11, Q12, Q2, Q3, Q4, Q7, Q8: MMBT2222, SamacSys_Parts:SOT95P240X114-3N, symbol SamacSys_Parts:MMBT2222
- added Q13, Q5, Q6: MMBT2907A-7-F, SOT96P240X100-3N, symbol SamacSys_Parts:MMBT2907A-7-F
- added R1, R10, R18, R19, R2, R20, R3, R9: 5.6k, Resistor_SMD:R_0402_1005Metric, symbol Device:R
- added R11, R14, R17, R33, R34, R35, R36, R37, R38, R39, R40, R41, R42, R43, R44, R45, R46, R5, R6: 100, Resistor_SMD:R_0402_1005Metric, symbol Device:R
- added R16: 5.1k, Resistor_SMD:R_0402_1005Metric, symbol Device:R
- added R31, R32: 1k, Resistor_SMD:R_0402_1005Metric, symbol Device:R
- added U2: BAT-HLD-001-TR, SamacSys_Parts:BATHLD001TR, symbol SamacSys_Parts:BAT-HLD-001-TR
- C1: value 1u -> .1u
- C2: value .01u -> .1u
- R12: value 1k -> 100
- R13: value 10k -> 100
- R15: value 5.6k -> 100
- R21, R23: value 100 -> 5.6k
- R26: value 100 -> 5.1k
- R27, R28: value 100 -> 10k
Connections:
- net +3V0: now also C1.1, C2.1, Q9.2, R24.1, R29.2, C14.1, C16.1, C18.1, C19.1, C20.1, C21.1, C22.1, C23.1, C24.1, C25.1, C26.1, C27.1, C28.1, C29.1, C30.1, C31.1, C4.1, C5.1, C9.1, IC11.5 (VCC), IC12.3 (IN0), IC12.5 (VCC), IC3.5 (VCC), IC5.5 (VCC), IC8.4 (RESET), IC8.8 (VDD), IC9.2 (1~{R}), IC9.4 (VCC), IC9.6 (2~{R}), Q1.3, Q2.3, Q4.3, Q5.2, Q6.2, R31.2; no longer Q10.2
- net +5V: now also C7.2, IC6.1 (INPUT)
- net 3V before switch: now also D10.1, D9.1
- net Button A: now also R23.1, R27.2, R8.1, C10.1, C12.1, IC3.1 (A), IC5.1 (B), R1.1, R18.2, R20.1, R3.1; no longer IC4.1 (A), R13.2
- net Button B: now also IC4.1 (A), R21.1, R28.2, C11.1, C13.1, IC5.2 (A), R10.1, R19.1, R2.1, R9.1; no longer R15.1, R8.1
- net CLK: now also R30.1, IC8.3 (OUT), IC9.1 (1~{CP}), IC9.5 (2~{CP})
- net GND: now also R26.1, R27.1, R28.1, C10.2, C11.2, C12.2, C13.2, C14.2, C15.2, C16.2, C17.2, C18.2, C19.2, C20.2, C21.2, C22.2, C23.2, C24.2, C25.2, C26.2, C27.2, C28.2, C29.2, C30.2, C31.2, C4.2, C5.2, C6.2, C7.1, C8.2, C9.2, D1.1 (K), D13.1 (K), D14.1 (K), D15.1 (K), D16.1 (K), D17.1 (K), D18.1 (K), D19.1 (K), D20.1 (K), D4.1 (K), D6.1 (K), IC11.2 (GND), IC12.2 (GND), IC3.3 (GND), IC5.3 (GND), IC6.2 (GROUND), IC8.1 (GND), IC9.11 (GND), Q11.2, Q12.2, Q13.3, Q8.2, R16.1, U2.3; no longer D12.1 (K), Q9.3, R13.1
- net at D2.2 (A): now also R6.1
- net at IC2.12 (1Q): now also R13.2
- net at J1.A5 (CC1): now also R16.2
- net at J1.B5 (CC2): now also R26.2
- net at IC4.2 (B): now also R15.2, IC3.4 (Y)
- net at VR1.3 (CW): now also C15.1, IC8.2 (TRIG), IC8.6 (THRES); no longer C1.1
- net at D8.2 (A): now also R17.2
- net at U3.4 (Y): now also IC9.10 (2K), IC9.7 (2J), R33.2
- net at IC4.4 (Y): now also IC3.2 (B), R14.2
- net at R12.1: now also D4.2 (A)
- net at IC13.15 (A0), IC14.15 (A0), IC15.15 (A0)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: now also IC10.6 (C), IC9.12 (1Q), R37.2; no longer R21.2
- net at U3.1 (A): now also IC11.6 (C), IC9.13 (1~{Q}); no longer IC10.6 (C)
- net at IC13.14 (A1), IC14.14 (A1), IC15.14 (A1)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: now also IC11.1 (A), IC9.9 (2Q), R36.2; no longer IC10.1 (A)
- net at IC10.3 (B), IC13.13 (A2), IC14.13 (A2)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: now also IC11.3 (B), R35.2
- net at IC14.6 (D): now also R44.1; no longer R28.1
- net at D7.2 (A): now also R15.1
- net at R8.2: now also Q7.1
- net at VR1.2 (WIPER): now also R32.2; no longer R12.2
- net at R25.1: now also IC5.4 (Y); no longer IC20.6 (D)
- net at DS1.17 (K_N), DS1.7 (K_T): now also R41.2; no longer R25.2
- net at IC16.6 (D): now also R46.1; no longer R30.1
- net at IC10.4 (Y): now also IC12.1 (IN1)
- net at R7.2: now also Q5.1
- net at IC19.6 (D): now also R40.1; no longer R24.1
- net at IC15.6 (D): now also R45.1; no longer R29.1
- net at DS1.13 (K_D): now also R45.2; no longer R29.2
- net at U1.4 (Y): now also R17.1
- net at IC13.6 (D): now also R43.1; no longer R27.1
- net at DS1.1 (K_A), DS1.18 (K_B): now also R43.2; no longer R27.2
- net at Q9.1: now also R18.1
- net at D11.2 (A): now also R22.1
- net at IC21.6 (D): now also R39.1; no longer R23.1
- net at DS1.5 (K_U): now also R39.2; no longer R23.2
- net at IC18.6 (D): now also R42.1; no longer R26.1
- net at R4.2: now also Q3.1
- net at DS1.14 (K_R), DS1.3 (K_K): now also R42.2; no longer R26.2
- net at D5.2 (A): now also R13.1
- net at Q10.1: now also R21.2
- net at Q10.3: now also R22.2, Q11.3, Q12.3
- net at IC17.6 (D): now also R38.1; no longer R22.1
- net at DS1.10 (K_E), DS1.15 (K_P), DS1.9 (K_F): now also R46.2; no longer R30.2
- net at DS1.16 (K_C): now also R44.2; no longer R28.2
- net at DS1.2 (K_M), DS1.6 (K_S): now also R40.2; no longer R24.2
- net at DS1.4 (K_H), DS1.8 (K_G): now also R38.2; no longer R22.2
- net at IC1.5 (Q): now also R11.1
- net at D3.2 (A): now also R11.2
- net at D12.2 (A): now also R24.2; no longer R21.1
- new net: IC10.1 (A), IC9.8 (2~{Q})
- new net: Q6.1, R9.2
- new net: IC11.4 (Y), IC12.6 (IN2)
- new net: D9.2, U2.1
- new net: Q8.1, R10.2
- new net: Q1.1, R2.2
- new net: IC8.7 (DISCH), R31.1, R32.1
- new net: Q3.2, R6.2
- new net: Q2.2, Q3.3
- new net: Q10.2, Q9.3
- new net: C17.1, IC8.5 (CONT)
- new net: Q11.1, R20.2
- new net: D17.2 (A), R34.1
- new net: D13.2 (A), R25.2
- new net: IC12.4 (Y), IC9.14 (1J), IC9.3 (1K), R34.2
- new net: D1.2 (A), R5.1
- new net: Q1.2, Q4.2, R5.2
- new net: D16.2 (A), R33.1
- new net: Q7.2, Q8.3
- new net: Q5.3, Q6.3, Q7.3, R12.2
- new net: IC20.6 (D), R41.1
- new net: Q2.1, R3.2
- new net: D20.2 (A), R37.1
- new net: Q13.1, R23.2
- new net: D15.2 (A), R30.2
- new net: D18.2 (A), R35.1
- new net: C6.1, C8.1, D10.2, IC6.3 (OUTPUT)
- new net: D19.2 (A), R36.1
- new net: Q12.1, R19.2
- new net: D12.1 (K), Q13.2
- new net: D14.2 (A), R29.1
- new net: Q4.1, R1.2
- new net: D6.2 (A), R14.1

Commit message: oops I didn't change the right schematic
Parts:
- removed D10, D9: LSM115JE3_TR13, SamacSys_Parts:DIOM5436X330N, symbol SamacSys_Parts:LSM115JE3_TR13
- removed D5, D6: LED, LED_SMD:LED_0402_1005Metric, symbol Device:LED
- removed IC10, IC11: SN74LVC1G11MDCKREP, SamacSys_Parts:SOP65P210X110-6N, symbol SamacSys_Parts:SN74LVC1G11MDCKREP
- removed IC12: SN74LVC1G97QDBVRQ1, SamacSys_Parts:SOT95P280X145-6N, symbol SamacSys_Parts:SN74LVC1G97QDBVRQ1
- removed IC20, IC21: TMUX1208QRSVRQ1, SamacSys_Parts:TMUX1208QRSVRQ1, symbol SamacSys_Parts:TMUX1208QRSVRQ1
- removed IC5: 74AUP1T87GWH, SOT65P212X110-5N, symbol SamacSys_Parts:74AUP1T87GWH
- removed IC6: NCV4274CDT33RKG, NCV4274CDT33RKG, symbol SamacSys_Parts:NCV4274CDT33RKG
- removed IC8: TLC555QDRQ1, SamacSys_Parts:SOIC127P600X175-8N, symbol SamacSys_Parts:TLC555QDRQ1
- removed IC9: 74HC73D,653, SamacSys_Parts:SOIC127P600X175-14N, symbol SamacSys_Parts:74HC73D,653
- removed Q10, Q5, Q6, Q9: MMBT2907A-7-F, SOT96P240X100-3N, symbol SamacSys_Parts:MMBT2907A-7-F
- removed Q11, Q12, Q7, Q8: MMBT2222, SamacSys_Parts:SOT95P240X114-3N, symbol SamacSys_Parts:MMBT2222
- removed U1: 74AHC1G86W5-7, SOT95P285X130-5N, symbol SamacSys_Parts:74AHC1G86W5-7
- removed U2: BAT-HLD-001-TR, SamacSys_Parts:BATHLD001TR, symbol SamacSys_Parts:BAT-HLD-001-TR
- removed U3: NC7S08M5X, SOT95P280X145-5N, symbol SamacSys_Parts:NC7S08M5X
- added D10, D9: LED, LED_SMD:LED_0402_1005Metric, symbol Device:LED
- added D5, D6: LSM115JE3_TR13, SamacSys_Parts:DIOM5436X330N, symbol SamacSys_Parts:LSM115JE3_TR13
- added IC10: 74AUP1G32GW-Q100H, SOT65P212X110-5N, symbol SamacSys_Parts:74AUP1G32GW-Q100H
- added IC11, IC12: TMUX1208QRSVRQ1, SamacSys_Parts:TMUX1208QRSVRQ1, symbol SamacSys_Parts:TMUX1208QRSVRQ1
- added IC20: TLC555QDRQ1, SamacSys_Parts:SOIC127P600X175-8N, symbol SamacSys_Parts:TLC555QDRQ1
- added IC21: 74AUP1T87GWH, SOT65P212X110-5N, symbol SamacSys_Parts:74AUP1T87GWH
- added IC5: NCV4274CDT33RKG, NCV4274CDT33RKG, symbol SamacSys_Parts:NCV4274CDT33RKG
- added IC6: 74HC73D,653, SamacSys_Parts:SOIC127P600X175-14N, symbol SamacSys_Parts:74HC73D,653
- added IC8, IC9: SN74LVC1G11MDCKREP, SamacSys_Parts:SOP65P210X110-6N, symbol SamacSys_Parts:SN74LVC1G11MDCKREP
- added Q10, Q5, Q6, Q9: PMV100EPAR, SOT95P230X110-3N, symbol SamacSys_Parts:PMV100EPAR
- added Q11, Q12, Q7, Q8: 2N7002_HAMR, 2N7002HAMR, symbol SamacSys_Parts:2N7002_HAMR
- added U1: BAT-HLD-001-TR, SamacSys_Parts:BATHLD001TR, symbol SamacSys_Parts:BAT-HLD-001-TR
- added U2: NC7S08M5X, SOT95P280X145-5N, symbol SamacSys_Parts:NC7S08M5X
- added U3: 74AHC1G86W5-7, SOT95P285X130-5N, symbol SamacSys_Parts:74AHC1G86W5-7
- C10, C11, C15: value 1u -> .1u
- C17: value .01u -> .1u
- C27, C8, C9: value .1u -> 1u
- C28: value .1u -> .01u
- C5: value .1u -> 10u
- C6: value 10u -> 100n
- C7: value 100n -> .1u
- R1, R10, R18, R19, R2, R20, R21, R23, R3, R4, R9: value 5.6k -> 100
- R16: value 5.1k -> 100
- R25: value 100 -> 1k
- R26: value 5.1k -> 1k
- R27, R28: value 10k -> 5.6k
- R29, R30, R33, R34, R35, R36, R39, R40, R41, R42, R44: value 100 -> 5.6k
- R31, R32: value 1k -> 100
- R5, R6: value 100 -> 5.1k
- R7, R8: value 5.6k -> 10k
Connections:
- net +3V0: now also C12.1, C13.1, C15.1, C17.1, IC13.4 (S3), IC14.10 (S5), IC14.2 (S1), IC14.3 (S2), IC15.10 (S5), IC15.3 (S2), IC16.4 (S3), IC16.9 (S6), IC17.5 (S4), IC19.10 (S5), IC19.3 (S2), IC7.6 (2~{R}), R25.2, R45.1, R9.2, IC10.5 (VCC), IC11.10 (S5), IC11.11 (VDD), IC11.16 (EN), IC11.2 (S1), IC11.3 (S2), IC11.5 (S4), IC12.11 (VDD), IC12.16 (EN), IC12.4 (S3), IC20.4 (RESET), IC20.8 (VDD), IC21.5 (VCC), IC6.14 (1J), IC6.2 (1~{R}), IC6.3 (1K), IC6.4 (VCC), IC8.5 (VCC), IC9.5 (VCC), Q5.3, Q6.3, Q9.3, U2.5 (VCC), U3.5 (VCC); no longer C27.1, C28.1, C5.1, C9.1, IC13.10 (S5), IC13.3 (S2), IC13.5 (S4), IC14.4 (S3), IC16.10 (S5), IC16.2 (S1), IC16.3 (S2), IC17.10 (S5), IC17.2 (S1), IC17.3 (S2), IC17.4 (S3), IC18.4 (S3), IC19.5 (S4), IC7.14 (1J), IC7.3 (1K), R24.1, R29.2, R31.2
- net +5V: now also C6.2, IC5.1 (INPUT); no longer C7.2
- net 3V before switch: now also D5.1, D6.1
- net Button A: now also C8.1, R27.1, R29.1, R33.1, R34.1, R39.2, R41.1, R44.1, R7.2, IC21.1 (B), U3.1 (A); no longer C12.1, R1.1, R18.2, R20.1, R23.1, R27.2, R3.1, R7.1, R8.1
- net Button B: now also C9.1, R28.1, R30.1, R35.1, R36.1, R40.1, R42.1, R8.2, IC21.2 (A), U3.2 (B); no longer C13.1, R10.1, R19.1, R2.1, R21.1, R28.2, R4.1, R9.1
- net CLK: now also IC7.5 (2~{CP}), R24.1, IC20.3 (OUT), IC6.1 (1~{CP}); no longer R30.1
- net GND: now also C6.1, C7.2, D12.1 (K), IC13.10 (S5), IC13.3 (S2), IC13.5 (S4), IC14.4 (S3), IC16.10 (S5), IC16.2 (S1), IC16.3 (S2), IC17.10 (S5), IC17.2 (S1), IC17.3 (S2), IC17.4 (S3), IC18.4 (S3), IC19.5 (S4), R5.1, R6.1, R7.1, R8.1, D10.1 (K), D9.1 (K), IC10.3 (GND), IC11.12 (GND), IC11.4 (S3), IC11.7 (S8), IC11.8 (S7), IC11.9 (S6), IC12.10 (S5), IC12.12 (GND), IC12.2 (S1), IC12.3 (S2), IC12.5 (S4), IC12.7 (S8), IC12.8 (S7), IC12.9 (S6), IC20.1 (GND), IC21.3 (GND), IC5.2 (GROUND), IC6.11 (GND), IC8.2 (GND), IC9.2 (GND), Q11.2, Q12.2, Q8.2, U1.3, U2.3 (GND), U3.3 (GND); no longer C6.2, C7.1, D19.1 (K), IC13.4 (S3), IC14.10 (S5), IC14.2 (S1), IC14.3 (S2), IC15.10 (S5), IC15.3 (S2), IC16.4 (S3), IC16.9 (S6), IC17.5 (S4), IC19.10 (S5), IC19.3 (S2), R16.1, R26.1, R27.1, R28.1
- net at IC13.13 (A2), IC14.13 (A2), IC15.13 (A2)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: now also R12.2, IC11.13 (A2), IC12.13 (A2), IC6.12 (1Q), IC8.3 (B), IC9.3 (B), U2.2 (B); no longer IC7.12 (1Q), R35.2
- net at IC13.15 (A0), IC14.15 (A0), IC15.15 (A0)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: now also IC7.12 (1Q), R14.2, IC11.15 (A0), IC12.15 (A0), IC8.6 (C); no longer R37.2
- net at IC7.10 (2K): now also IC7.7 (2J), R10.2, U2.4 (Y)
- net at IC7.13 (1~{Q}): now also IC9.6 (C), U2.1 (A)
- net at IC7.8 (2~{Q}): now also IC8.1 (A)
- net at IC7.9 (2Q): now also IC13.14 (A1), IC14.14 (A1), IC15.14 (A1), IC16.14 (A1), IC17.14 (A1), IC18.14 (A1), IC19.14 (A1), R13.2, IC11.14 (A1), IC12.14 (A1), IC9.1 (A)
- net at J1.A5 (CC1): now also R5.2; no longer R16.2
- net at R39.1: now also Q9.1
- net at DS1.5 (K_U): now also R16.2; no longer R39.2
- net at R2.2: now also IC2.12 (1Q); no longer Q1.1
- net at R31.1: now also D14.2 (A); no longer R32.1
- net at R32.2: now also Q3.2; no longer VR1.2 (WIPER)
- net at D8.2 (A): now also R10.1; no longer R17.2
- net at Q3.1: now also R30.2; no longer R4.2
- net at R6.2: now also J1.B5 (CC2); no longer Q3.2
- net at R22.1: now also IC13.6 (D); no longer D11.2 (A)
- net at R22.2: now also DS1.13 (K_D)
- net at IC15.6 (D): now also R15.1; no longer R45.1
- net at R21.2: now also DS1.16 (K_C)
- net at VR1.3 (CW): now also C27.1, IC20.2 (TRIG), IC20.6 (THRES); no longer C15.1
- net at R20.2: now also DS1.1 (K_A), DS1.18 (K_B)
- net at IC14.6 (D): now also R23.1; no longer R44.1
- net at R44.2: now also Q13.1; no longer DS1.16 (K_C)
- net at D17.2 (A): now also R38.2; no longer R34.1
- net at IC3.2 (B), IC4.4 (Y): now also R3.2; no longer R14.2
- net at IC3.4 (Y), IC4.2 (B): now also R4.2; no longer R15.2
- net at D4.2 (A): now also R4.1; no longer R12.1
- net at R13.1: now also D11.2 (A)
- net at D2.2 (A): now also R2.1; no longer R6.1
- net at R25.1: now also R26.1, IC20.7 (DISCH)
- net at D13.2 (A): now also R24.2; no longer R25.2
- net at R34.2: now also Q7.1
- net at D1.2 (A): now also R1.2; no longer R5.1
- net at Q1.2, Q4.2: now also R31.2; no longer R5.2
- net at R18.1: now also IC18.6 (D)
- net at D16.2 (A): now also R37.1; no longer R33.1
- net at R33.2: now also Q5.1
- net at R38.1: now also U3.4 (Y); no longer IC17.6 (D)
- net at R45.2: now also D19.2 (A); no longer DS1.13 (K_D)
- net at R11.1: now also D9.2 (A); no longer IC1.5 (Q)
- net at R11.2: now also IC7.14 (1J), IC7.3 (1K), IC10.4 (Y); no longer D3.2 (A)
- net at D7.2 (A): now also R9.1; no longer R15.1
- net at R26.2: now also VR1.2 (WIPER); no longer J1.B5 (CC2)
- net at Q2.1: now also R29.2; no longer R3.2
- net at D20.2 (A): now also R46.2; no longer R37.1
- net at R23.2: now also DS1.10 (K_E), DS1.15 (K_P), DS1.9 (K_F); no longer Q13.1
- net at R43.1: now also D18.2 (A); no longer IC13.6 (D)
- net at D15.2 (A): now also R32.1; no longer R30.2
- net at IC19.6 (D): now also R16.1; no longer R40.1
- net at DS1.2 (K_M), DS1.6 (K_S): now also R17.2; no longer R40.2
- net at DS1.17 (K_N), DS1.7 (K_T): now also R18.2; no longer R41.2
- net at D12.2 (A): now also R14.1; no longer R24.2
- net at R19.2: now also DS1.14 (K_R), DS1.3 (K_K)
- net at Q13.2: now also D19.1 (K); no longer D12.1 (K)
- net at R17.1: now also IC17.6 (D)
- net at R46.1: now also IC21.4 (Y); no longer IC16.6 (D)
- net at DS1.4 (K_H), DS1.8 (K_G): now also R15.2; no longer R38.2
- net at Q4.1: now also R27.2; no longer R1.2
- new net: Q1.1, R28.2
- new net: Q5.2, Q6.2, Q7.3, R37.2
- new net: IC10.1 (B), IC8.4 (Y)
- new net: Q10.2, Q11.3, Q12.3, R43.2
- new net: Q12.1, R40.2
- new net: C5.1, C7.1, D6.2, IC5.3 (OUTPUT)
- new net: IC12.6 (D), R21.1
- new net: Q8.1, R36.2
- new net: Q7.2, Q8.3
- new net: Q10.1, R42.2
- new net: Q10.3, Q9.2
- new net: C28.1, IC20.5 (CONT)
- new net: IC1.5 (Q), R1.1
- new net: IC11.6 (D), R20.1
- new net: D10.2 (A), R12.1
- new net: IC10.2 (A), IC9.4 (Y)
- new net: D5.2, U1.1
- new net: Q6.1, R35.2
- new net: IC16.6 (D), R19.1
- new net: D3.2 (A), R3.1
- new net: Q11.1, R41.2
Other:
- note added: "CMOS NAND Gate"
- note added: "CMOS NOR Gate"
- note removed: "NAND Gate"
- note removed: "NOR Gate"
