File: Logic-PCB/Logic-PCB.kicad_pcb (KiCad board)
At the start: 2 copper layers, 118 parts, among them IC1 74LVC1G74DC-Q100H, IC10 SN74LVC1G11MDCKREP, IC11 SN74LVC1G11MDCKREP, IC12 SN74LVC1G97QDBVRQ1, IC13 SN74LVC1G97QDBVRQ1, IC14 TMUX1208QRSVRQ1, IC15 TMUX1208QRSVRQ1, IC16 TMUX1208QRSVRQ1, IC17 TMUX1208QRSVRQ1, IC18 TMUX1208QRSVRQ1, IC19 TMUX1208QRSVRQ1, IC2 74HC73D,653, IC20 TMUX1208QRSVRQ1, IC21 TMUX1208QRSVRQ1, IC22 TMUX1208QRSVRQ1, IC3 SN74LVC1G02DBVR, IC4 SN74LVC1G02DBVR, IC5 NCV4274AST33T3G, IC6 74AUP1T87GWH, IC7 74HC73D,653, IC8 TLC555QDRQ1, IC9 74HC73D,653, J1 CX70M-24P1, Q1 MMBT2222, Q10 MMBT2907A-7-F, Q11 MMBT2222, Q12 MMBT2222, Q13 MMBT2907A-7-F, Q2 MMBT2222, Q3 MMBT2222, Q4 MMBT2222, Q5 MMBT2907A-7-F, Q6 MMBT2907A-7-F, Q7 MMBT2222, Q8 MMBT2222, Q9 MMBT2907A-7-F, SW1 SW_Push, SW2 SW_Push, SW3 SW_Push, U1 74AHC1G86W5-7, U2 BAT-HLD-001-TR

Commit message: updates from meeting
Parts:
- removed IC13: SN74LVC1G97QDBVRQ1, SamacSys_Parts:SOT95P280X145-6N
- removed IC5: NCV4274AST33T3G, SamacSys_Parts:SOT230P700X175-4N
- removed R16, R32, R5, R6: 10k, Resistor_SMD:R_0402_1005Metric
- removed SW3: SW_Push, SamacSys_Parts:SKPMBHE010
- added C10: .1u, Capacitor_SMD:C_01005_0402Metric, F.Cu at (99.3, 139.7)
- added C11: .1u, Capacitor_SMD:C_01005_0402Metric, F.Cu at (107.9, 139.7)
- added C12: .1u, Capacitor_SMD:C_01005_0402Metric, F.Cu at (108.7, 151.1)
- added C13: .1u, Capacitor_SMD:C_01005_0402Metric, F.Cu at (108.7, 142.7)
- added C14: .1u, Capacitor_SMD:C_01005_0402Metric, F.Cu at (103.4, 150.9)
- added C15: .1u, Capacitor_SMD:C_01005_0402Metric, F.Cu at (103.5, 143.6)
- added C16: .1u, Capacitor_SMD:C_01005_0402Metric, F.Cu at (117.2, 137.2)
- added C17: .1u, Capacitor_SMD:C_01005_0402Metric, F.Cu at (122.5, 137.2)
- added C18: .1u, Capacitor_SMD:C_01005_0402Metric, F.Cu at (127.9, 137.2)
- added C19: .1u, Capacitor_SMD:C_01005_0402Metric, F.Cu at (117.2, 143.3)
- added C20: .1u, Capacitor_SMD:C_01005_0402Metric, F.Cu at (122.5, 143.3)
- added C21: .1u, Capacitor_SMD:C_01005_0402Metric, F.Cu at (127.9, 143.3)
- added C22: .1u, Capacitor_SMD:C_01005_0402Metric, F.Cu at (117.3, 149.5)
- added C23: .1u, Capacitor_SMD:C_01005_0402Metric, F.Cu at (122.5, 149.5)
- added C24: .1u, Capacitor_SMD:C_01005_0402Metric, F.Cu at (127.8, 149.5)
- added C25: .1u, Capacitor_SMD:C_01005_0402Metric, F.Cu at (92.5, 115.6)
- added C26: .1u, Capacitor_SMD:C_01005_0402Metric, F.Cu at (92.1, 123.4)
- added C27: .1u, Capacitor_SMD:C_01005_0402Metric, F.Cu at (144.0, 49.5)
- added C30: 1u, Capacitor_SMD:C_01005_0402Metric, F.Cu at (84.7, 48.3)
- added C31: .1u, Capacitor_SMD:C_01005_0402Metric, F.Cu at (90.4, 48.3)
- added C32: 1u, Capacitor_SMD:C_01005_0402Metric, F.Cu at (95.5, 48.3)
- added C33: .1u, Capacitor_SMD:C_01005_0402Metric, F.Cu at (100.9, 48.3)
- added C6: .1u, Capacitor_SMD:C_01005_0402Metric, F.Cu at (133.0, 75.2)
- added C7: .1u, Capacitor_SMD:C_01005_0402Metric, F.Cu at (135.7, 91.4)
- added C8: .1u, Capacitor_SMD:C_01005_0402Metric, F.Cu at (134.6, 101.0)
- added C9: .1u, Capacitor_SMD:C_01005_0402Metric, F.Cu at (134.6, 109.0)
- added D20: LSM115JE3_TR13, SamacSys_Parts:DIOM5436X330N, F.Cu at (139.1, 43.3)
- added IC23: NCV4274CDT33RKG, SamacSys_Parts:NCV4274CDT33RKG, F.Cu at (153.5, 45.8)
- added U3: NC7S08M5X, SamacSys_Parts:SOT95P280X145-5N, F.Cu at (108.7, 149.0)
- R1, R2: value 10k -> 5.1k
- moved R2 77.2 mm to (137.4, 30.1), turned to 90 degrees
- moved R1 74.8 mm to (156.7, 30.2), turned to 90 degrees
- moved D9 37.4 mm to (106.2, 41.5)
- moved U2 4.35 mm to (122.7, 38.4)
- moved D11 3.59 mm to (102.9, 56.3), turned to 90 degrees
- moved R28 3.08 mm to (98.8, 56.2), turned to 90 degrees
- moved J1 2.24 mm to (147.1, 33.8)
- moved R27 2.12 mm to (93.9, 56.2), turned to 90 degrees
Connections:
- C1 pad 1: +3V0 -> GND
- C2 pad 1: 3V before switch -> Net-(IC23-OUTPUT)
- C2 pad 2: +3V0 -> GND
- C3 pad 2: +3V0 -> GND
- C4 pad 2: +3V0 -> GND
- C5 pad 2: +3V0 -> GND
- D1 pad 1: +3V0 -> GND
- D10 pad 1: +3V0 -> GND
- D12 pad 1: +3V0 -> GND
- D13 pad 1: +3V0 -> GND
- D14 pad 1: +3V0 -> GND
- D15 pad 1: +3V0 -> GND
- D16 pad 1: +3V0 -> GND
- D17 pad 1: +3V0 -> GND
- D18 pad 1: +3V0 -> GND
- D19 pad 1: +3V0 -> GND
- D2 pad 1: +3V0 -> GND
- D3 pad 1: +3V0 -> GND
- D4 pad 1: +3V0 -> GND
- D5 pad 1: +3V0 -> GND
- D6 pad 1: +3V0 -> GND
- D7 pad 1: +3V0 -> GND
- D8 pad 1: +3V0 -> GND
- DS1 pad 11: +3V0 -> GND
- DS1 pad 12: +3V0 -> GND
- IC1 pad 4: +3V0 -> GND
- IC10 pad 2: +3V0 -> GND
- IC11 pad 2: +3V0 -> GND
- IC12 pad 2: +3V0 -> GND
- IC14 pad 12: +3V0 -> GND
- IC14 pad 4: +3V0 -> GND
- IC14 pad 7: +3V0 -> GND
- IC14 pad 8: +3V0 -> GND
- IC14 pad 9: +3V0 -> GND
- IC15 pad 10: +3V0 -> GND
- IC15 pad 12: +3V0 -> GND
- IC15 pad 2: +3V0 -> GND
- IC15 pad 3: +3V0 -> GND
- IC15 pad 5: +3V0 -> GND
- IC15 pad 7: +3V0 -> GND
- IC15 pad 8: +3V0 -> GND
- IC15 pad 9: +3V0 -> GND
- IC16 pad 10: +3V0 -> GND
- IC16 pad 12: +3V0 -> GND
- IC16 pad 3: +3V0 -> GND
- IC16 pad 5: +3V0 -> GND
- IC16 pad 7: +3V0 -> GND
- IC16 pad 8: +3V0 -> GND
- IC16 pad 9: +3V0 -> GND
- IC17 pad 12: +3V0 -> GND
- IC17 pad 4: +3V0 -> GND
- IC17 pad 5: +3V0 -> GND
- IC17 pad 7: +3V0 -> GND
- IC17 pad 8: +3V0 -> GND
- IC17 pad 9: +3V0 -> GND
- IC18 pad 12: +3V0 -> GND
- IC18 pad 5: +3V0 -> GND
- IC18 pad 7: +3V0 -> GND
- IC18 pad 8: +3V0 -> GND
- IC18 pad 9: +3V0 -> GND
- IC19 pad 10: +3V0 -> GND
- IC19 pad 12: +3V0 -> GND
- IC19 pad 2: +3V0 -> GND
- IC19 pad 3: +3V0 -> GND
- IC19 pad 5: +3V0 -> GND
- IC19 pad 7: +3V0 -> GND
- IC19 pad 8: +3V0 -> GND
- IC2 pad 11: +3V0 -> GND
- IC20 pad 10: +3V0 -> GND
- IC20 pad 12: +3V0 -> GND
- IC20 pad 2: +3V0 -> GND
- IC20 pad 3: +3V0 -> GND
- IC20 pad 4: +3V0 -> GND
- IC20 pad 7: +3V0 -> GND
- IC20 pad 8: +3V0 -> GND
- IC20 pad 9: +3V0 -> GND
- IC21 pad 10: +3V0 -> GND
- IC21 pad 12: +3V0 -> GND
- IC21 pad 2: +3V0 -> GND
- IC21 pad 3: +3V0 -> GND
- IC21 pad 4: +3V0 -> GND
- IC21 pad 5: +3V0 -> GND
- IC21 pad 7: +3V0 -> GND
- IC21 pad 8: +3V0 -> GND
- IC22 pad 12: +3V0 -> GND
- IC22 pad 2: +3V0 -> GND
- IC22 pad 4: +3V0 -> GND
- IC22 pad 5: +3V0 -> GND
- IC22 pad 7: +3V0 -> GND
- IC22 pad 8: +3V0 -> GND
- IC22 pad 9: +3V0 -> GND
- IC3 pad 3: +3V0 -> GND
- IC4 pad 3: +3V0 -> GND
- IC6 pad 3: +3V0 -> GND
- IC7 pad 1: Button -> CLK
- IC7 pad 11: +3V0 -> GND
- IC8 pad 1: +3V0 -> GND
- IC9 pad 1: Button -> CLK
- IC9 pad 11: +3V0 -> GND
- IC9 pad 5: Button -> CLK
- J1 pad A1: +3V0 -> GND
- J1 pad A12: +3V0 -> GND
- J1 pad A5: unconnected-(J1-CC1-PadA5) -> Net-(J1-CC1)
- J1 pad B1: +3V0 -> GND
- J1 pad B12: +3V0 -> GND
- J1 pad B5: unconnected-(J1-CC2-PadB5) -> Net-(J1-CC2)
- Q11 pad 2: +3V0 -> GND
- Q12 pad 2: +3V0 -> GND
- Q13 pad 3: +3V0 -> GND
- Q8 pad 2: +3V0 -> GND
- R1 pad 1: +3V0 -> GND
- R1 pad 2: Button A -> Net-(J1-CC2)
- R2 pad 1: +3V0 -> GND
- R2 pad 2: Button B -> Net-(J1-CC1)
- R30 pad 1: +3V0 -> GND
- R31 pad 1: +3V0 -> GND
- S1 pad 3: +3V0 -> GND
- S1 pad 7: +3V0 -> GND
- U1 pad 3: +3V0 -> GND
- U2 pad 3: +3V0 -> GND

Commit message: CMOS
Parts:
- moved DS1 0.27 mm to (139.3, 129.4)
Changed lines of the file:
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@@
   )
   (footprint "SamacSys_Parts:PSA0811GWA" (layer "F.Cu")
-    (at 139.11 129.54)
+    (at 139.344 129.413)
     (descr "PSA08-11GWA-1")
     (tags "Display")
