File: Logic-PCB/Logic-PCB.kicad_pcb (KiCad board)
At the start: 2 copper layers, 148 parts, among them IC1 74LVC1G74DC-Q100H, IC10 SN74LVC1G11MDCKREP, IC11 SN74LVC1G11MDCKREP, IC12 74AUP1G32GW-Q100H, IC13 TMUX1208QRSVRQ1, IC14 TMUX1208QRSVRQ1, IC15 TMUX1208QRSVRQ1, IC16 TMUX1208QRSVRQ1, IC17 TMUX1208QRSVRQ1, IC18 TMUX1208QRSVRQ1, IC19 TMUX1208QRSVRQ1, IC2 74HC73D,653, IC20 TMUX1208QRSVRQ1, IC21 TMUX1208QRSVRQ1, IC3 SN74LVC1G02DBVR, IC4 SN74LVC1G02DBVR, IC5 74AUP1T87GWH, IC6 NCV4274CDT33RKG, IC7 74HC73D,653, IC8 TLC555QDRQ1, IC9 74HC73D,653, J1 CX70M-24P1, Q1 BC847,215, Q10 PMV100EPAR, Q11 2N7002_HAMR, Q12 2N7002_HAMR, Q13 BC858B,235, Q2 BC847,215, Q3 BC847,215, Q4 BC847,215, Q5 PMV100EPAR, Q6 PMV100EPAR, Q7 2N7002_HAMR, Q8 2N7002_HAMR, Q9 PMV100EPAR, SW1 SW_Push, SW2 SW_Push, U1 74AHC1G86W5-7, U3 NC7S08M5X

Commit message: Layout
Parts:
- removed J1: CX70M-24P1, SamacSys_Parts:CX70M24P1
- added D21: LED, LED_SMD:LED_0402_1005Metric, F.Cu at (95.3, 68.9)
- added D9: LED, LED_SMD:LED_0402_1005Metric, F.Cu at (95.3, 51.2)
- added R47: 100, Resistor_SMD:R_0402_1005Metric, F.Cu at (91.9, 52.2)
- added R48: 100, Resistor_SMD:R_0402_1005Metric, F.Cu at (83.5, 69.9)
- added U2: ~, Connector:USB-C UJC-HP-G-5-SMT-TR, F.Cu at (143.3, 82.8)
- moved IC7 39.0 mm to (105.7, 69.9), turned to 0 degrees
- moved C8 3.78 mm to (129.8, 81.3), turned to 180 degrees
- moved C6 2.63 mm to (129.8, 83.5), turned to 180 degrees
- moved R16 2.52 mm to (132.9, 84.7)
- moved R26 2.52 mm to (133.0, 82.3)
- moved C22 2.14 mm to (109.6, 75.8)
- moved C4 1.79 mm to (83.5, 66.8), turned to 90 degrees
- moved C7 1.79 mm to (129.8, 85.7), turned to 90 degrees
- moved D10 1.73 mm to (130.8, 76.9), turned to 0 degrees
- moved IC1 1.13 mm to (81.5, 68.5), turned to 90 degrees
- moved R14 0.64 mm to (88.5, 87.5), turned to 180 degrees
- moved R11 0.31 mm to (82.8, 60.8)
- moved R18 0.21 mm to (62.6, 64.3)
Connections:
- IC1 pad 3: unconnected-(IC1-~{Q}-Pad3) -> Net-(IC1-~{Q})
- IC2 pad 13: unconnected-(IC2-1~{Q}-Pad13) -> Net-(IC2-1~{Q})
Routing:
- net +3V0: track 627.5 -> 668.7 mm, vias 6 -> 7
- net CLK: track 161.6 -> 126.9 mm
- net +5V: track 52.9 -> 29.2 mm
- net Net-(U2-CC1): track 21.7 -> 3.53 mm
- net GND: track 27.0 -> 44.4 mm, vias 5 -> 19
- net Net-(IC10-Y): track 16.3 -> 28.8 mm
- net Net-(IC2-1~{Q}): track 0.00 -> 12.4 mm
- net Net-(D21-A): track 0.00 -> 11.8 mm
- net Net-(IC11-A): track 124.1 -> 135.1 mm
- net Net-(U2-CC2): track 9.40 -> 2.95 mm
- net Net-(IC1-Q): track 10.9 -> 6.15 mm
- net Net-(IC10-B): track 173.3 -> 177.9 mm, vias 8 -> 10
- net Net-(IC6-OUTPUT): track 18.1 -> 14.1 mm
- net Net-(D9-A): track 0.00 -> 3.79 mm
- net Net-(IC1-~{Q}): track 0.00 -> 3.08 mm
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
Commit message: Layout
Parts:
- added G***: LOGO, Logic:Gentex Logo, F.Cu at (122.4, 21.1)
- added G***: LOGO, Logic:Calvin Logo, F.Cu at (88.6, 19.8)
Routing:
- net GND: track 44.4 -> 57.9 mm
Other:
- board outline added: 127.3 x 76.5 mm
- board text removed: "GENTEX | Calvin University"

Commit message: layout
Routing:
- net Button B: track 262.4 -> 261.6 mm
Changed lines of the file:
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@@
   (segment (start 61.74 48.5) (end 61.74 55.2) (width 0.15) (layer "F.Cu") (net 46))
   (segment (start 42.87 64.67) (end 37.599828 64.67) (width 0.15) (layer "F.Cu") (net 46))
+  (segment (start 88.44 73.62) (end 94.31 73.62) (width 0.15) (layer "F.Cu") (net 46))
   (segment (start 33.99 83.59) (end 34.82 84.42) (width 0.15) (layer "F.Cu") (net 46))
+  (segment (start 87.58 74.48) (end 88.44 73.62) (width 0.15) (layer "F.Cu") (net 46))
   (segment (start 31.3 32.66) (end 34.08 32.66) (width 0.15) (layer "F.Cu") (net 46))
   (segment (start 33.6 65.96) (end 33.6 66.94) (width 0.15) (layer "F.Cu") (net 46))
   (segment (start 69.905026 60.18) (end 67.205 60.18) (width 0.15) (layer "F.Cu") (net 46))
+  (segment (start 85.515 79.535) (end 85.515 76.545) (width 0.15) (layer "F.Cu") (net 46))
   (segment (start 86.39 79.66) (end 85.64 79.66) (width 0.15) (layer "F.Cu") (net 46))
   (segment (start 43.9 77.24) (end 43.9 82.28) (width 0.15) (layer "F.Cu") (net 46))
   (segment (start 33.735 65.825) (end 33.6 65.96) (width 0.15) (layer "F.Cu") (net 46))
-  (segment (start 87.06 73.64) (end 94.29 73.64) (width 0.15) (layer "F.Cu") (net 46))
   (segment (start 66.79 58.16) (end 66.33 57.7) (width 0.15) (layer "F.Cu") (net 46))
   (segment (start 34.08 34.3) (end 34.08 32.66) (width 0.15) (layer "F.Cu") (net 46))
@@
   (segment (start 67.205 60.18) (end 66.79 59.765) (width 0.15) (layer "F.Cu") (net 46))
   (segment (start 58.38 82.28) (end 59.055 82.28) (width 0.15) (layer "F.Cu") (net 46))
-  (segment (start 85.515 75.185) (end 87.06 73.64) (width 0.15) (layer "F.Cu") (net 46))
   (segment (start 43.56 61.08) (end 43.56 63.98) (width 0.15) (layer "F.Cu") (net 46))
   (segment (start 61.74 47.09) (end 61.74 48.5) (width 0.15) (layer "F.Cu") (net 46))
@@
   (segment (start 85.84 55.694974) (end 85.84 51.002) (width 0.15) (layer "F.Cu") (net 46))
   (segment (start 36.48 60.29) (end 42.77 60.29) (width 0.15) (layer "F.Cu") (net 46))
+  (segment (start 94.31 73.62) (end 96.78 71.15) (width 0.15) (layer "F.Cu") (net 46))
   (segment (start 43.9 82.28) (end 43.48 82.7) (width 0.15) (layer "F.Cu") (net 46))
-  (segment (start 85.515 79.535) (end 85.515 75.185) (width 0.15) (layer "F.Cu") (net 46))
   (segment (start 35.052 81.976) (end 34.414 81.976) (width 0.15) (layer "F.Cu") (net 46))
   (segment (start 43.56 63.98) (end 42.87 64.67) (width 0.15) (layer "F.Cu") (net 46))
@@
   (segment (start 34.414 81.976) (end 33.99 82.4) (width 0.15) (layer "F.Cu") (net 46))
   (segment (start 42.97 43.23) (end 42.54 42.8) (width 0.15) (layer "F.Cu") (net 46))
+  (segment (start 85.515 76.545) (end 87.58 74.48) (width 0.15) (layer "F.Cu") (net 46))
   (segment (start 34.495 47.325) (end 35.4 46.42) (width 0.15) (layer "F.Cu") (net 46))
   (segment (start 34.985 65.825) (end 33.735 65.825) (width 0.15) (layer "F.Cu") (net 46))
@@
   (segment (start 59.18 72.595) (end 65.115 66.66) (width 0.15) (layer "F.Cu") (net 46))
   (segment (start 87.125026 56.98) (end 85.84 55.694974) (width 0.15) (layer "F.Cu") (net 46))
-  (segment (start 94.29 73.64) (end 96.78 71.15) (width 0.15) (layer "F.Cu") (net 46))
-  (via (at 87.06 73.64) (size 0.8) (drill 0.4) (layers "F.Cu" "B.Cu") (net 46))
-  (via (at 59.18 73.64) (size 0.8) (drill 0.4) (layers "F.Cu" "B.Cu") (net 46))
-  (segment (start 87.06 73.64) (end 87.06 73.13) (width 0.15) (layer "B.Cu") (net 46))
-  (segment (start 59.18 73.27) (end 59.18 73.64) (width 0.15) (layer "B.Cu") (net 46))
-  (segment (start 59.71 72.74) (end 59.18 73.27) (width 0.15) (layer "B.Cu") (net 46))
-  (segment (start 87.06 73.13) (end 86.67 72.74) (width 0.15) (layer "B.Cu") (net 46))
-  (segment (start 86.67 72.74) (end 59.71 72.74) (width 0.15) (layer "B.Cu") (net 46))
+  (via (at 87.58 74.48) (size 0.8) (drill 0.4) (layers "F.Cu" "B.Cu") (net 46))
+  (via (at 59.18 74.48) (size 0.8) (drill 0.4) (layers "F.Cu" "B.Cu") (net 46))
+  (segment (start 87.57 74.48) (end 86.78 73.69) (width 0.25) (layer "B.Cu") (net 46))
+  (segment (start 87.58 74.48) (end 87.57 74.48) (width 0.25) (layer "B.Cu") (net 46))
+  (segment (start 59.97 73.69) (end 59.18 74.48) (width 0.25) (layer "B.Cu") (net 46))
+  (segment (start 86.78 73.69) (end 59.97 73.69) (width 0.25) (layer "B.Cu") (net 46))
   (segment (start 89.29 85.610172) (end 88.370172 86.53) (width 0.15) (layer "F.Cu") (net 47))
   (segment (start 87.52 80.1) (end 89.29 81.87) (width 0.15) (layer "F.Cu") (net 47))
@@
   (segment (start 112.84 40.82) (end 112.84 40.27) (width 0.15) (layer "F.Cu") (net 111))
   (segment (start 123.4 59.97) (end 123 59.97) (width 0.15) (layer "F.Cu") (net 111))
-  (segment (start 105.76 77.05) (end 103.13 77.05) (width 0.15) (layer "F.Cu") (net 111))
   (segment (start 106.74 45.54) (end 106.74 45.14) (width 0.15) (layer "F.Cu") (net 111))
   (segment (start 106.74 38.11) (end 106.34 38.11) (width 0.15) (layer "F.Cu") (net 111))
@@
   (segment (start 114.64 59.63) (end 115.19 59.63) (width 0.15) (layer "F.Cu") (net 111))
   (segment (start 105.34 38.86) (end 105.34 39.51) (width 0.15) (layer "F.Cu") (net 111))
-  (segment (start 103.13 77.05) (end 99.72 73.64) (width 0.15) (layer "F.Cu") (net 111))
   (segment (start 106.74 46.34) (end 106.74 46.72) (width 0.15) (layer "F.Cu") (net 111))
   (segment (start 121.26 70.29) (end 121.66 69.89) (width 0.15) (layer "F.Cu") (net 111))
@@
   (segment (start 114.24 49.45) (end 114.04 49.25) (width 0.15) (layer "F.Cu") (net 111))
   (segment (start 105.34 45.89) (end 105.34 46.54) (width 0.15) (layer "F.Cu") (net 111))
+  (segment (start 105.76 77.05) (end 102.29 77.05) (width 0.15) (layer "F.Cu") (net 111))
   (segment (start 106.74 59.2) (end 106.74 59.6) (width 0.15) (layer "F.Cu") (net 111))
   (segment (start 105.84 43.775025) (end 105.84 42.94) (width 0.15) (layer "F.Cu") (net 111))
@@
   (segment (start 113.64 49.25) (end 114.04 49.25) (width 0.15) (layer "F.Cu") (net 111))
   (segment (start 104.94 59) (end 104.94 58.48) (width 0.15) (layer "F.Cu") (net 111))
+  (segment (start 102.29 77.05) (end 99.72 74.48) (width 0.15) (layer "F.Cu") (net 111))
   (segment (start 106.14 51.97) (end 106.14 53.57) (width 0.15) (layer "F.Cu") (net 111))
   (segment (start 122.775 57.995) (end 122.8 58.02) (width 0.15) (layer "F.Cu") (net 111))
@@
   (segment (start 104.94 44.38) (end 104.47 43.91) (width 0.15) (layer "F.Cu") (net 111))
   (segment (start 106.74 38.51) (end 106.74 38.11) (width 0.15) (layer "F.Cu") (net 111))
-  (via (at 79.14 73.64) (size 0.8) (drill 0.4) (layers "F.Cu" "B.Cu") (free) (net 111))
-  (via (at 111.92 73.88) (size 0.8) (drill 0.4) (layers "F.Cu" "B.Cu") (free) (net 111))
+  (via (at 79.14 74.48) (size 0.8) (drill 0.4) (layers "F.Cu" "B.Cu") (free) (net 111))
+  (via (at 111.92 74.48) (size 0.8) (drill 0.4) (layers "F.Cu" "B.Cu") (free) (net 111))
   (via (at 114.25 69.1) (size 0.8) (drill 0.4) (layers "F.Cu" "B.Cu") (free) (net 111))
   (via (at 109.61 81.47) (size 0.8) (drill 0.4) (layers "F.Cu" "B.Cu") (free) (net 111))
   (via (at 123.81 77.49) (size 0.8) (drill 0.4) (layers "F.Cu" "B.Cu") (free) (net 111))
-  (via (at 84.29 73.64) (size 0.8) (drill 0.4) (layers "F.Cu" "B.Cu") (free) (net 111))
+  (via (at 84.29 74.48) (size 0.8) (drill 0.4) (layers "F.Cu" "B.Cu") (free) (net 111))
   (via (at 99.72 81.47) (size 0.8) (drill 0.4) (layers "F.Cu" "B.Cu") (free) (net 111))
   (via (at 99.72 62.89) (size 0.8) (drill 0.4) (layers "F.Cu" "B.Cu") (free) (net 111))
@@
   (via (at 85.61 56.98) (size 0.8) (drill 0.4) (layers "F.Cu" "B.Cu") (free) (net 111))
   (via (at 59.18 20.23) (size 0.8) (drill 0.4) (layers "F.Cu" "B.Cu") (free) (net 111))
-  (via (at 99.72 73.64) (size 0.8) (drill 0.4) (layers "F.Cu" "B.Cu") (free) (net 111))
-  (via (at 60.87 73.64) (size 0.8) (drill 0.4) (layers "F.Cu" "B.Cu") (free) (net 111))
+  (via (at 99.72 74.48) (size 0.8) (drill 0.4) (layers "F.Cu" "B.Cu") (free) (net 111))
+  (via (at 60.87 74.48) (size 0.8) (drill 0.4) (layers "F.Cu" "B.Cu") (free) (net 111))
   (via (at 59.18 55.58) (size 0.8) (drill 0.4) (layers "F.Cu" "B.Cu") (free) (net 111))
   (via (at 111.59 69.09) (size 0.8) (drill 0.4) (layers "F.Cu" "B.Cu") (free) (net 111))
