File: Logic-PCB/_autosave-Logic-PCB.kicad_sch (KiCad schematic)
At the start: 144 parts, among them IC1 74LVC1G74DC-Q100H, IC10 74AUP1G32GW-Q100H, IC11 TMUX1208QRSVRQ1, IC12 TMUX1208QRSVRQ1, IC13 TMUX1208QRSVRQ1, IC14 TMUX1208QRSVRQ1, IC15 TMUX1208QRSVRQ1, IC16 TMUX1208QRSVRQ1, IC17 TMUX1208QRSVRQ1, IC18 TMUX1208QRSVRQ1, IC19 TMUX1208QRSVRQ1, IC2 74HC73D,653, IC20 TLC555QDRQ1, IC21 74AUP1T87GWH, IC3 SN74LVC1G02DBVR, IC4 SN74LVC1G02DBVR, IC5 NCV4274CDT33RKG, IC6 74HC73D,653, IC7 74HC73D,653, IC8 SN74LVC1G11MDCKREP, IC9 SN74LVC1G11MDCKREP, Q1 BC847,215, Q10 PMV100EPAR, Q11 2N7002_HAMR, Q12 2N7002_HAMR, Q13 BC858B,235, Q2 BC847,215, Q3 BC847,215, Q4 BC847,215, Q5 PMV100EPAR, Q6 PMV100EPAR, Q7 2N7002_HAMR, Q8 2N7002_HAMR, Q9 PMV100EPAR, SW1 SW_Push, SW2 SW_Push, U1 BAT-HLD-001-TR, U2 NC7S08M5X, U3 74AHC1G86W5-7

Commit message: Layout
Parts:
- U2: footprint (none) -> Connector:USB-C UJC-HP-G-5-SMT-TR
Changed lines of the file:
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@@
       (effects (font (size 1.27 1.27)))
     )
-    (property "Footprint" "" (at 143.256 81.28 0)
+    (property "Footprint" "Connector:USB-C UJC-HP-G-5-SMT-TR" (at 143.256 81.28 0)
       (effects (font (size 1.27 1.27)) hide)
     )
